File: Hardware/SparkFun_Thing_Plus_NORA_W306.sch (EAGLE design)
At the start: 72 parts, among them J1 THING_PLUS_LOGICAL, J2 LiPo, J3 QWIIC_RA, J4 MICRO-SDFRICTION, J5 USB-C, J6 SWD (DNP), Q1 3.1A/30V/105mΩ, Q2 MBT3904DW1T1, U1 UBLOX_NORA_W306, U3 XC6222B331MR-G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

Commit message: Pre-group Review of v04 Changes
-moved logos to right box in SCH
-added column names to may pin mapping table in SCH
-adjusted SCH note about boot strapping pin internal pullups
-"single-cell" lipo batt note moved to single line
-changed current jumper silk to be "CUR"
-changed MEAS to smaller size and flat ends to fit better
-Adjusted V_BATT trace on inner layer to be 90 degreees when crossing the I2C lines
-Nudges trace off of user button for better gnd flow, added via nearby
-Added GND trace off of GND pad on fuel guage IC
-Nudges I2C vias near Fuel guage IC for better ground flow. added gnd vias nearby
-Nudges trace under charge IC for better gnd flow
-Larger SFE logo on top silk
-Larger OSHW logo on back
-Larger product name text on bottom silk
-updated NORA-w306 trestrict to rectangels rather than polys
-added silk lines to help populate close small passives
Parts:
- LOGO2: value OSHW-LOGOMINI -> OSHW-LOGOM; device SparkFun-Aesthetics:OSHW-LOGOMINI -> SparkFun-Aesthetics:OSHW-LOGOM
Other:
- note added: "***Boot Strap Pins*** (W306 includes internal pull-ups) See DS PG 10 for more info. PA30 PB19/SWD_DATA PA7/UART-LOG-TXD"
- note added: "ARDUINO"
- note added: "MODULE"
- note added: "V_BATT should be a single-cell LiPo battery."
- note removed: "***Boot Strap Pins*** (Include internal pull-ups) See DS PG 10 for more info. PA30 PB19/SWD_DATA PA7/UART-LOG-TXD"
- note removed: "V_BATT should be a single- cell LiPo battery."
- moved on the sheet: C4, J6, U1
