File: Hardware/Production/SparkFun_Thing_Plus_NORA_W306-Panel.brd (EAGLE design)
At the start: 130 x 141.7 mm, 1506 parts, among them J1 THING_PLUS_LOGICAL, J10 THING_PLUS_LOGICAL, J11 MICRO-SDFRICTION, J12 SWD (DNP), J13 LiPo, J14 QWIIC_RA, J15 USB-C, J16 THING_PLUS_LOGICAL, J17 MICRO-SDFRICTION, J18 SWD (DNP), J19 LiPo, J2 LiPo, J20 QWIIC_RA, J21 USB-C, J22 THING_PLUS_LOGICAL, J23 MICRO-SDFRICTION, J24 SWD (DNP), J25 LiPo, J26 QWIIC_RA, J27 USB-C, J28 THING_PLUS_LOGICAL, J29 MICRO-SDFRICTION, J3 QWIIC_RA, J30 SWD (DNP), J31 LiPo, J32 QWIIC_RA, J33 USB-C, J34 THING_PLUS_LOGICAL, J35 MICRO-SDFRICTION, J36 SWD (DNP), J37 LiPo, J38 QWIIC_RA, J39 USB-C, J4 MICRO-SDFRICTION, J40 THING_PLUS_LOGICAL, J41 MICRO-SDFRICTION, J42 SWD (DNP), J43 LiPo, J44 QWIIC_RA, J45 USB-C, J46 THING_PLUS_LOGICAL, J47 MICRO-SDFRICTION, J48 SWD (DNP), J49 LiPo, J5 USB-C, J50 QWIIC_RA, J51 USB-C, J52 THING_PLUS_LOGICAL, J53 MICRO-SDFRICTION, J54 SWD (DNP), J55 LiPo, J56 QWIIC_RA, J57 USB-C, J58 THING_PLUS_LOGICAL, J59 MICRO-SDFRICTION, J6 SWD (DNP), J60 SWD (DNP), J7 LiPo, J8 QWIIC_RA, J9 USB-C, Q1 3.1A/30V/105mΩ, Q10 MBT3904DW1T1, Q11 3.1A/30V/105mΩ, Q12 MBT3904DW1T1, Q13 3.1A/30V/105mΩ, Q14 MBT3904DW1T1, Q15 3.1A/30V/105mΩ, Q16 MBT3904DW1T1, Q17 3.1A/30V/105mΩ, Q18 MBT3904DW1T1, Q19 3.1A/30V/105mΩ, Q2 MBT3904DW1T1, Q20 MBT3904DW1T1, Q3 3.1A/30V/105mΩ, Q4 MBT3904DW1T1, Q5 3.1A/30V/105mΩ, Q6 MBT3904DW1T1, Q7 3.1A/30V/105mΩ, Q8 MBT3904DW1T1, Q9 3.1A/30V/105mΩ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

Commit message: proto panel v04
Parts:
- removed C100, C109, C112, C113, C122, C125, C126, C44, C47, C48, C57, C60, C61, C70, C73, C74, C83, C86, C87, C96, C99: 10uF, SparkFun-Capacitors:0402-TIGHT
- removed C101, C102, C103, C104, C110, C114, C115, C116, C117, C123, C127, C128, C129, C130, C37, C38, C39, C45, C49, C50, C51, C52, C58, C62, C63, C64, C65, C71, C75, C76, C77, C78, C84, C88, C89, C90, C91, C97: 0.1uF, SparkFun-Capacitors:0402-TIGHT
- removed C105, C106, C118, C119, C40, C41, C53, C54, C66, C67, C79, C80, C92, C93: 1.0uF, SparkFun-Capacitors:0402-TIGHT
- removed C107, C108, C111, C120, C121, C124, C42, C43, C46, C55, C56, C59, C68, C69, C72, C81, C82, C85, C94, C95, C98: 4.7uF, SparkFun-Capacitors:0603
- removed CHG3, CHG4, CHG5, CHG6, CHG7, CHG8, CHG9, JP10, JP11, JP12, JP13, JP14, JP15, JP16, JP17, JP18, JP19, JP20, JP21, JP22, JP23, JP24, JP25, JP26, JP27, JP28, JP29, JP30, JP31, JP32, JP33, JP34, JP35, JP36, JP37, JP38, JP39, JP40, LED3, LED4, LED5, LED6, LED7, LED8, LED9, USBSHLD3, USBSHLD4, USBSHLD5, USBSHLD6, USBSHLD7, USBSHLD8, USBSHLD9: (no value), SparkFun-Jumpers:SMT-JUMPER_2_NC_TRACE_SILK
- removed CUR3, CUR4, CUR5, CUR6, CUR7, CUR8, CUR9: (no value), SparkFun-Jumpers:SMT-JUMPER_3_1-NC_TRACE_SILK
- removed D19, D25, D31, D37, D43, D49, D55: 1A/23V/620mV, SparkFun-DiscreteSemi:SOD-323
- removed D20, D26, D32, D38, D44, D50, D56: Yellow, SparkFun-LED:LED-0603
- removed D21, D27, D33, D39, D45, D51, D57: BLUE, SparkFun-LED:LED-0603
- removed D22, D28, D34, D40, D46, D52, D58: RED, SparkFun-LED:LED-0603
- removed D23, D29, D35, D41, D47, D53, D59: PRTR5V0U2F, SparkFun-IC-Power:SOT886
- removed D24, D30, D36, D42, D48, D54, D60: WS2812, SparkFun-LED:WS2812-2020
- removed E1, E10, E2, E3, E4, E5, E6, E7, E8, E9: SPH0641LM4H-1, SparkFun-Sensors:SPH0641LM4H-1_MICROPHONE
- removed FD13, FD14, FD15, FD16, FD17, FD18, FD19, FD20, FD21, FD22, FD23, FD24, FD25, FD26, FD27, FD28, FD29, FD30, FD31, FD32, FD33, FD34, FD35, FD36, FD37, FD38, FD39, FD40: FIDUCIALUFIDUCIAL, SparkFun-Aesthetics:FIDUCIAL-MICRO
- removed H13, H14, H15, H16, H17, H18, H19, H20, H21, H22, H23, H24, H25, H26, H27, H28, H29, H30, H31, H32, H33, H34, H35, H36, H37, H38, H39, H40: STAND-OFF, SparkFun-Hardware:STAND-OFF
- removed I2C3, I2C4, I2C5, I2C6, I2C7, I2C8, I2C9: JUMPER-SMT_3_2-NC_TRACE_SILK, SparkFun-Jumpers:SMT-JUMPER_3_2-NC_TRACE_SILK
- removed J19, J25, J31, J37, J43, J49, J55: LiPo, SparkFun-Connectors:JST-2-SMD
- removed J20, J26, J32, J38, J44, J50, J56: QWIIC_RA, SparkFun-Connectors:JST04_1MM_RA
- removed J21, J27, J33, J39, J45, J51, J57: USB-C, SparkFun-Connectors:USB-C-16P-4LAYER-ISOLATED
- removed J22, J28, J34, J40, J46, J52, J58: THING_PLUS_LOGICAL, SparkFun-Boards:THING_PLUS
- removed J23, J29, J35, J41, J47, J53, J59: MICRO-SDFRICTION, SparkFun-Connectors:MICROSD_TINY
- removed J24, J30, J36, J42, J48, J54, J60: SWD (DNP), SparkFun-Connectors:2X5-SMD-UNSHROUDED
- removed LOGO10, LOGO13, LOGO16, LOGO19, LOGO22, LOGO25, LOGO28: OSHW-LOGOMINI, SparkFun-Aesthetics:OSHW-LOGO-MINI
- removed LOGO11, LOGO14, LOGO17, LOGO20, LOGO23, LOGO26, LOGO29: QWIIC_LOGO_4MM, SparkFun-Aesthetics:QWIIC_4MM
- removed LOGO12, LOGO15, LOGO18, LOGO21, LOGO24, LOGO27, LOGO30: SFE_LOGO_NAME_FLAME.1_INCH, SparkFun-Aesthetics:SFE_LOGO_NAME_FLAME_.1
- removed Q16, Q18, Q20: MBT3904DW1T1, SparkFun-DiscreteSemi:SC70-6
- removed Q17, Q19: 3.1A/30V/105mΩ, SparkFun-DiscreteSemi:SOT23-3
- removed R100, R117, R118, R135, R136, R153, R154, R171, R172, R81, R82, R99: 5.1k, SparkFun-Resistors:0402-TIGHT
- removed R101, R104, R105, R109, R112, R119, R122, R123, R127, R130, R137, R140, R141, R145, R148, R155, R158, R159, R163, R166, R173, R176, R177, R76, R83, R86, R87, R91, R94: 10k, SparkFun-Resistors:0402-TIGHT
- removed R102, R120, R138, R156, R174, R84: 100, SparkFun-Resistors:0402-TIGHT
- removed R103, R106, R121, R124, R139, R142, R157, R160, R175, R178, R85, R88: 1k, SparkFun-Resistors:0402-TIGHT
- removed R107, R108, R125, R126, R143, R144, R161, R162, R179, R180, R89, R90: 2.2k, SparkFun-Resistors:0402-TIGHT
- removed R110, R113, R128, R131, R146, R149, R164, R167, R77, R92, R95: 4.7k, SparkFun-Resistors:0402-TIGHT
- removed R111, R129, R147, R165, R93: 2.0k, SparkFun-Resistors:0603
- removed R114, R132, R150, R168, R78, R96: 100k, SparkFun-Resistors:0402-TIGHT
- removed R115, R133, R151, R169, R79, R97: 22k, SparkFun-Resistors:0402-TIGHT
- removed R116, R134, R152, R170, R80, R98: 33k, SparkFun-Resistors:0402-TIGHT
- removed S10, S13, S16, S19, S22, S25, S28: RESET, SparkFun-Switches:TACTILE_SWITCH_SMD_4.6X2.8MM
- removed S11, S14, S17, S20, S23, S26, S29: BOOT, SparkFun-Switches:TACTILE_SWITCH_SMD_4.6X2.8MM
- removed S12, S15, S18, S21, S24, S27, S30: USER, SparkFun-Switches:TACTILE_SWITCH_SMD_4.6X2.8MM
- removed TP1, TP10, TP2, TP3, TP4, TP5, TP6, TP7, TP8, TP9: TEST-POINT3X5, SparkFun-Connectors:PAD.03X.05
- removed U$259, U$334, U$409, U$484, U$559, U$634, U$709: (no value), output:#15#15
- removed U$260, U$335, U$410, U$485, U$560, U$635, U$710: (no value), output:#16#16
- removed U$261, U$336, U$411, U$486, U$561, U$636, U$711: (no value), output:1417
- removed U$262, U$337, U$412, U$487, U$562, U$637, U$712: (no value), output:#9#91420
- removed U$263, U$338, U$413, U$488, U$563, U$638, U$713: (no value), output:#10#91420
- removed U$264, U$339, U$414, U$489, U$564, U$639, U$714: (no value), output:#11#91420
- removed U$265, U$340, U$415, U$490, U$565, U$640, U$715: (no value), output:#12#91420
- removed U$266, U$341, U$416, U$491, U$566, U$641, U$716: (no value), output:#13#91420
- removed U$267, U$342, U$417, U$492, U$567, U$642, U$717: (no value), output:#14#91420
- removed U$268, U$343, U$418, U$493, U$568, U$643, U$718: (no value), output:#15#91420
- removed U$269, U$344, U$419, U$494, U$569, U$644, U$719: (no value), output:#16#91420
- removed U$270, U$345, U$420, U$495, U$570, U$645, U$720: (no value), output:#8#91421
- removed U$271, U$346, U$421, U$496, U$571, U$646, U$721: (no value), output:#7#8
- removed U$272, U$347, U$422, U$497, U$572, U$647, U$722: (no value), output:#6#8
- removed U$273, U$348, U$423, U$498, U$573, U$648, U$723: (no value), output:#5#8
- removed U$274, U$349, U$424, U$499, U$574, U$649, U$724: (no value), output:#4#8
- removed U$275, U$350, U$425, U$500, U$575, U$650, U$725: (no value), output:#3#8
- removed U$276, U$351, U$426, U$501, U$576, U$651, U$726: (no value), output:#2#8
- removed U$277, U$352, U$427, U$502, U$577, U$652, U$727: (no value), output:#1#8
- removed U$278, U$353, U$428, U$503, U$578, U$653, U$728: (no value), output:#0#8
- removed U$279, U$354, U$429, U$504, U$579, U$654, U$729: (no value), output:#SHLD#9
- removed U$280, U$355, U$430, U$505, U$580, U$655, U$730: (no value), output:#GND#10
- removed U$281, U$356, U$431, U$506, U$581, U$656, U$731: (no value), output:#CHG#13
- removed U$282, U$357, U$432, U$507, U$582, U$657, U$732: (no value), output:#PWR#14
- removed U$283, U$358, U$433, U$508, U$583, U$658, U$733: (no value), output:#JP1#18
- removed U$284, U$359, U$434, U$509, U$584, U$659, U$734: (no value), output:#JP2#18
- removed U$285, U$360, U$435, U$510, U$585, U$660, U$735: (no value), output:#A0#18
- removed U$286, U$361, U$436, U$511, U$586, U$661, U$736: (no value), output:#A1#18
- removed U$287, U$362, U$437, U$512, U$587, U$662, U$737: (no value), output:#A2#18
- removed U$288, U$363, U$438, U$513, U$588, U$663, U$738: (no value), output:#G#18
- removed U$289, U$364, U$439, U$514, U$589, U$664, U$739: (no value), output:#JP3#0
- removed U$290, U$365, U$440, U$515, U$590, U$665, U$740: (no value), output:16165
- removed U$291, U$366, U$441, U$516, U$591, U$666, U$741: (no value), output:USER0
- removed U$292, U$367, U$442, U$517, U$592, U$667, U$742: (no value), output:##RESET##0
- removed U$293, U$368, U$443, U$518, U$593, U$668, U$743: (no value), output:#NC#1
- removed U$294, U$369, U$444, U$519, U$594, U$669, U$744: (no value), output:#NC#2
- removed U$295, U$370, U$445, U$520, U$595, U$670, U$745: (no value), output:#I2C#3
- removed U$296, U$371, U$446, U$521, U$596, U$671, U$746: (no value), output:#JP4#0
- removed U$297, U$372, U$447, U$522, U$597, U$672, U$747: (no value), output:RGB_155
- removed U$298, U$373, U$448, U$523, U$598, U$673, U$748: (no value), output:#500#501
- removed U$299, U$374, U$449, U$524, U$599, U$674, U$749: (no value), output:#100#501
- removed U$300, U$375, U$450, U$525, U$600, U$675, U$750: (no value), output:#SWD#501
- removed U$301, U$307, U$376, U$382, U$451, U$457, U$526, U$532, U$601, U$607, U$676, U$682: (no value), output:CHG0
- removed U$302, U$377, U$452, U$527, U$602, U$677: (no value), output:RESET0
- removed U$303, U$378, U$453, U$528, U$603, U$678: (no value), output:#VUSB#0
- removed U$304, U$379, U$454, U$529, U$604, U$679: (no value), output:#VBAT#0
- removed U$305, U$380, U$455, U$530, U$605, U$680: (no value), output:#EN#0
- removed U$306, U$381, U$456, U$531, U$606, U$681: (no value), output:#3V3#0
- removed U$308, U$383, U$458, U$533, U$608, U$683: (no value), output:MA0
- removed U$309, U$311, U$384, U$386, U$459, U$461, U$534, U$536, U$609, U$611, U$684, U$686: (no value), output:THING_PLUS_0
- removed U$310, U$385, U$460, U$535, U$610, U$685: (no value), output:BOOT0
- removed U$312, U$387, U$462, U$537, U$612, U$687: (no value), output:PWR0
- removed U$313, U$314, U$388, U$389, U$463, U$464, U$538, U$539, U$613, U$614, U$688, U$689: (no value), output:NORA#W3060
- removed U$315, U$390, U$465, U$540, U$615, U$690: (no value), SparkFun-Aesthetics:SFE_LOGO_FLAME_.1
- removed U$316, U$391, U$466, U$541, U$616, U$691: (no value), output:#A0#1
- removed U$317, U$392, U$467, U$542, U$617, U$692: (no value), output:#A1#1
- removed U$318, U$393, U$468, U$543, U$618, U$693: (no value), output:#A2#4
- removed U$319, U$394, U$469, U$544, U$619, U$694: (no value), output:#0#4
- removed U$320, U$395, U$470, U$545, U$620, U$695: (no value), output:#1#4
- removed U$321, U$396, U$471, U$546, U$621, U$696: (no value), output:#2#CS#5
- removed U$322, U$397, U$472, U$547, U$622, U$697: (no value), output:#3#SCK#5
- removed U$323, U$398, U$473, U$548, U$623, U$698: (no value), output:#4#PICO#5
- removed U$324, U$399, U$474, U$549, U$624, U$699: (no value), output:#5#POCI#5
- removed U$325, U$400, U$475, U$550, U$625, U$700: (no value), output:#6#RX1#6
- removed U$326, U$401, U$476, U$551, U$626, U$701: (no value), output:#7#TX1#7
- removed U$327, U$402, U$477, U$552, U$627, U$702: (no value), output:#8#8
- removed U$328, U$403, U$478, U$553, U$628, U$703: (no value), output:#SDA#9#10
- removed U$329, U$404, U$479, U$554, U$629, U$704: (no value), output:#SCL#10#10
- removed U$330, U$405, U$480, U$555, U$630, U$705: (no value), output:#11#11
- removed U$331, U$406, U$481, U$556, U$631, U$706: (no value), output:#12#12
- removed U$332, U$407, U$482, U$557, U$632, U$707: (no value), output:#13#13
- removed U$333, U$408, U$483, U$558, U$633, U$708: (no value), output:#14#14
- removed U16, U21, U26, U31, U36, U41, U46: MCP73831, SparkFun-IC-Power:SOT23-5
- removed U17, U22, U27, U32, U37, U42, U47: XC6222B331MR-G, SparkFun-IC-Power:SOT23-5
- removed U18, U23, U28, U33, U38, U43, U48: UBLOX_NORA_W306, nora-w306:UBLOX-NORA-W3
- removed U19, U24, U29, U34, U39, U44, U49: MAX17048, SparkFun-IC-Power:DFN-8
- removed U20, U25, U30, U35, U40, U45, U50: CP2102N_QFN28, nora-w306:QFN28
- added MEAS, MEAS1, MEAS2: (no value), SparkFun-Jumpers:COMBO-JUMPER_2_NC_TRACE
- added SDPC, SDPC1, SDPC2: (no value), SparkFun-Jumpers:SMT-JUMPER_3_1-NC_TRACE_SILK
- C13, C27, C28: value 1.0uF -> 4.7uF; device SparkFun-Capacitors:0402-TIGHT -> SparkFun-Capacitors:0603
- C16, C20, C29, C33: value 4.7uF -> 10uF; device SparkFun-Capacitors:0603 -> SparkFun-Capacitors:0402-TIGHT
- C17, C22, C34, C35: value 10uF -> 0.1uF
- C18: value 0.1uF -> 4.7uF; device SparkFun-Capacitors:0402-TIGHT -> SparkFun-Capacitors:0603
- C25, C26, C9: value 0.1uF -> 1.0uF
- C30: value 4.7uF -> 0.1uF; device SparkFun-Capacitors:0603 -> SparkFun-Capacitors:0402-TIGHT
- C31: value 10uF -> 4.7uF; device SparkFun-Capacitors:0402-TIGHT -> SparkFun-Capacitors:0603
- C32: value 0.1uF -> 10uF
- J11, J17, J4: value MICRO-SDFRICTION -> SDFRICTION
- J12, J18, J6: device SparkFun-Connectors:2X5-SMD-UNSHROUDED -> SparkFun-Connectors:2X5-SMD-UNSHROUDED_DNP_NO_PASTE
- LOGO1, LOGO2, LOGO7: value OSHW-LOGOMINI -> OSHW-LOGOM; device SparkFun-Aesthetics:OSHW-LOGO-MINI -> SparkFun-Aesthetics:OSHW-LOGO-M
- Q1, Q11, Q13, Q3, Q9: value 3.1A/30V/105mΩ -> 20V/4.2A/52mΩ/1.4W
- Q10: value MBT3904DW1T1 -> 20V/0.2A/8MHz/1.2Ω/1Vth; device SparkFun-DiscreteSemi:SC70-6 -> SparkFun-DiscreteSemi:SOT-416FL
- Q14, Q4, Q6, Q8: value MBT3904DW1T1 -> 20V/4.2A/52mΩ/1.4W; device SparkFun-DiscreteSemi:SC70-6 -> SparkFun-DiscreteSemi:SOT23-3
- Q15, Q5: value 3.1A/30V/105mΩ -> 20V/0.2A/8MHz/1.2Ω/1Vth; device SparkFun-DiscreteSemi:SOT23-3 -> SparkFun-DiscreteSemi:SOT-416FL
- Q7: value 3.1A/30V/105mΩ -> MBT3904DW1T1; device SparkFun-DiscreteSemi:SOT23-3 -> SparkFun-DiscreteSemi:SC70-6
- R14, R37, R50, R69, R73: value 10k -> 100
- R16, R56: value 4.7k -> 100k
- R19: value 2.0k -> 100k; device SparkFun-Resistors:0603 -> SparkFun-Resistors:0402-TIGHT
- R2, R52: value 1k -> 4.7k
- R20, R47: value 10k -> 100k
- R21: value 4.7k -> 100
- R22: value 100k -> 1k
- R23: value 22k -> 100
- R24: value 33k -> 10k
- R25: value 5.1k -> 4.7k
- R26: value 5.1k -> 2.0k; device SparkFun-Resistors:0402-TIGHT -> SparkFun-Resistors:0603
- R30, R66: value 100 -> 4.7k
- R31, R70: value 1k -> 100k
- R32: value 10k -> 22k
- R33, R58: value 10k -> 33k
- R34: value 1k -> 5.1k
- R35: value 2.2k -> 5.1k
- R36, R54: value 2.2k -> 10k
- R38, R74: value 4.7k -> 1k
- R39: value 2.0k -> 10k; device SparkFun-Resistors:0603 -> SparkFun-Resistors:0402-TIGHT
- R42: value 100k -> 2.2k
- R43: value 22k -> 2.2k
- R44, R62: value 33k -> 100
- R45, R46: value 5.1k -> 100k
- R53: value 2.2k -> 2.0k; device SparkFun-Resistors:0402-TIGHT -> SparkFun-Resistors:0603
- R55: value 10k -> 4.7k
- R57: value 2.0k -> 22k; device SparkFun-Resistors:0603 -> SparkFun-Resistors:0402-TIGHT
- R59: value 4.7k -> 5.1k
- R60: value 100k -> 5.1k
- R61: value 22k -> 10k
- R63: value 5.1k -> 1k
- R64: value 5.1k -> 10k
- R67: value 1k -> 2.2k
- R68: value 10k -> 2.2k
- R71, R72: value 2.2k -> 100k
- R75: value 2.0k -> 100; device SparkFun-Resistors:0603 -> SparkFun-Resistors:0402-TIGHT
- U$1: device output:#9#91420 -> output:#17#11
- U$10: device output:THING_PLUS_0 -> output:#GND#ON#3061714141842
- U$100: device output:#6#RX1#6 -> output:#1#4
- U$101: device output:#7#TX1#7 -> output:#13#13
- U$102: device output:#8#8 -> output:#14#14
- U$103: device output:#SDA#9#10 -> output:#15#15
- U$104: device output:#SCL#10#10 -> output:#16#16
- U$105: device output:#11#11 -> output:#11#91420
- U$106: device output:#12#12 -> output:#12#91420
- U$107: device output:#13#13 -> output:#13#91420
- U$108: device output:#14#14 -> output:#14#91420
- U$109: device output:#15#15 -> output:#15#91420
- U$110: device output:#16#16 -> output:#16#91420
- U$111: device output:1417 -> output:#8#91421
- U$112: device output:#9#91420 -> output:#7#8
- U$113: device output:#10#91420 -> output:#6#8
- U$114: device output:#11#91420 -> output:#5#8
- U$115: device output:#12#91420 -> output:#4#8
- U$116: device output:#13#91420 -> output:#3#8
- U$117: device output:#14#91420 -> output:#2#8
- U$118: device output:#15#91420 -> output:#1#8
- U$119: device output:#16#91420 -> output:#0#8
- U$120: device output:#8#91421 -> output:#SHLD#9
- U$121: device output:#7#8 -> output:#GND#10
- U$122: device output:#6#8 -> output:#CHG#13
- U$123: device output:#5#8 -> output:#PWR#14
- U$124: device output:#4#8 -> output:#A0#18
- U$125: device output:#3#8 -> output:USER0
- U$126: device output:#2#8 -> output:#NC#2
- U$127: device output:#1#8 -> output:#I2C#3
- U$128: device output:#0#8 -> output:#SWD#501
- U$129: device output:#SHLD#9 -> output:#JP2#0
- U$13: device output:#A1#1 -> output:#SDA#11#28
- U$130: device output:#GND#10 -> output:#LED_DO#0
- U$131: device output:#CHG#13 -> output:#JP1#0
- U$132: device output:#PWR#14 -> output:#9#10
- U$133: device output:#JP1#18 -> output:#10#11
- U$134: device output:#JP2#18 -> output:#17#11
- U$135: device output:#A0#18 -> output:#18#18
- U$136, U$68: device output:#A1#18 -> output:##RESET##19
- U$137, U$69: device output:#A2#18 -> output:#NC#21
- U$138: device output:#G#18 -> output:#G#22
- U$139: device output:#JP3#0 -> output:#3V#23
- U$14: device output:#A2#4 -> output:#17#28
- U$140: device output:16165 -> output:#VU#23
- U$141: device output:USER0 -> output:#VB26
- U$142: device output:##RESET##0 -> output:#EN#27
- U$143: device output:#NC#1 -> output:#2#28
- U$144: device output:#NC#2 -> output:#3#28
- U$145: device output:#I2C#3 -> output:#4#CS#28
- U$146: device output:#JP4#0 -> output:#5#SCK#28
- U$147: device output:RGB_155 -> output:#6#PICO#28
- U$148: device output:#500#501 -> output:#7#POCI#28
- U$149: device output:#100#501 -> output:#8#RX1#A1#28
- U$150: device output:#SWD#501 -> output:#9#TX1#A2#28
- U$151: device output:CHG0 -> output:#10#28
- U$152: device output:RESET0 -> output:#SDA#11#28
- U$153: device output:#VUSB#0 -> output:#SCL#12#28
- U$154: device output:#VBAT#0 -> output:#17#28
- U$155: device output:#EN#0 -> output:#18#28
- U$156: device output:#3V3#0 -> SparkFun-Aesthetics:SFE_LOGO_FLAME_.1
- U$157: device output:CHG0 -> output:#LD#29
- U$158: device output:MA0 -> output:1830
- U$159: device output:THING_PLUS_0 -> output:RGB_14141832
- U$160: device output:BOOT0 -> output:#VB26
- U$161: device output:THING_PLUS_0 -> output:CUR1714141837
- U$162: device output:PWR0 -> output:#MEAS#1714141838
- U$163: device output:NORA#W3060 -> output:THING_PLUS1714141839
- U$164: device output:NORA#W3060 -> output:NORA#W3061714141840
- U$165: device SparkFun-Aesthetics:SFE_LOGO_FLAME_.1 -> output:#GND#ON#3061714141842
- U$166: device output:#A0#1 -> output:23061714141843
- U$167: device output:#A1#1 -> output:#17#11
- U$168: device output:#A2#4 -> output:SDPC23061714141844
- U$169: device output:#0#4 -> output:##RST##23061714141845
- U$17: device output:#3#SCK#5 -> output:#SCL#12#28
- U$170: device output:#1#4 -> output:#JP3#23061714141846
- U$171: device output:#2#CS#5 -> output:#100#23061714141846
- U$172: device output:#3#SCK#5 -> output:#500#23061714141846
- U$173: device output:#4#PICO#5 -> output:CHG0
- U$174: device output:#5#POCI#5 -> output:RESET0
- U$175: device output:#6#RX1#6 -> output:#VUSB#0
- U$176: device output:#7#TX1#7 -> output:#EN#0
- U$177: device output:#8#8 -> output:#3V3#0
- U$178: device output:#SDA#9#10 -> output:MA0
- U$179: device output:#SCL#10#10 -> output:THING_PLUS_0
- U$18: device output:#4#PICO#5 -> output:#18#28
- U$180: device output:#11#11 -> output:BOOT0
- U$181: device output:#12#12 -> output:PWR0
- U$182: device output:#13#13 -> output:NORA#W3060
- U$183: device output:#14#14 -> SparkFun-Aesthetics:SFE_LOGO_FLAME_.2
- U$184: device output:#15#15 -> output:#A0#1
- U$185: device output:#16#16 -> output:#0#4
- U$186: device output:1417 -> output:#1#4
- U$187: device output:#9#91420 -> output:#13#13
- U$188: device output:#10#91420 -> output:#14#14
- U$189: device output:#11#91420 -> output:#15#15
- U$19: device output:#5#POCI#5 -> SparkFun-Aesthetics:SFE_LOGO_FLAME_.1
- U$190: device output:#12#91420 -> output:#16#16
- U$191: device output:#13#91420 -> output:#11#91420
- U$192: device output:#14#91420 -> output:#12#91420
- U$193: device output:#15#91420 -> output:#13#91420
- U$194: device output:#16#91420 -> output:#14#91420
- U$195: device output:#8#91421 -> output:#15#91420
- U$196: device output:#7#8 -> output:#16#91420
- U$197: device output:#6#8 -> output:#8#91421
- U$198: device output:#5#8 -> output:#7#8
- U$199: device output:#4#8 -> output:#6#8
- U$20: device output:#2#CS#5 -> output:#LD#29
- U$200: device output:#3#8 -> output:#5#8
- U$201: device output:#2#8 -> output:#4#8
- U$202: device output:#1#8 -> output:#3#8
- U$203: device output:#0#8 -> output:#2#8
- U$204: device output:#SHLD#9 -> output:#1#8
- U$205: device output:#GND#10 -> output:#0#8
- U$206: device output:#CHG#13 -> output:#SHLD#9
- U$207: device output:#PWR#14 -> output:#GND#10
- U$208: device output:#JP1#18 -> output:#CHG#13
- U$209: device output:#JP2#18 -> output:#PWR#14
- U$21: device output:#6#RX1#6 -> output:1830
- U$211: device output:#A1#18 -> output:USER0
- U$212: device output:#A2#18 -> output:#NC#2
- U$213: device output:#G#18 -> output:#I2C#3
- U$214: device output:#JP3#0 -> output:#SWD#501
- U$215: device output:16165 -> output:#JP2#0
- U$216: device output:USER0 -> output:#LED_DO#0
- U$217: device output:##RESET##0 -> output:#JP1#0
- U$218: device output:#NC#1 -> output:#9#10
- U$219: device output:#NC#2 -> output:#10#11
- U$22: device output:#7#TX1#7 -> output:#17#11
- U$220: device output:#I2C#3 -> output:#17#11
- U$221: device output:#JP4#0 -> output:#18#18
- U$222: device output:RGB_155 -> output:##RESET##19
- U$223: device output:#500#501 -> output:#NC#21
- U$224: device output:#100#501 -> output:#G#22
- U$225: device output:#SWD#501 -> output:#3V#23
- U$226: device output:CHG0 -> output:#VU#23
- U$227: device output:RESET0 -> output:#VB26
- U$228: device output:#VUSB#0 -> output:#EN#27
- U$229: device output:#VBAT#0 -> output:#2#28
- U$230: device output:#EN#0 -> output:#3#28
- U$231: device output:#3V3#0 -> output:#4#CS#28
- U$232: device output:CHG0 -> output:#5#SCK#28
- U$233: device output:MA0 -> output:#6#PICO#28
- U$234, U$86: device output:THING_PLUS_0 -> output:#7#POCI#28
- U$235: device output:BOOT0 -> output:#8#RX1#A1#28
- U$236: device output:THING_PLUS_0 -> output:#9#TX1#A2#28
- U$237: device output:PWR0 -> output:#10#28
- U$238: device output:NORA#W3060 -> output:#SDA#11#28
- U$239: device output:NORA#W3060 -> output:#SCL#12#28
- U$24: device output:#8#8 -> output:RGB_14141832
- U$240: device SparkFun-Aesthetics:SFE_LOGO_FLAME_.1 -> output:#17#28
- U$241: device output:#A0#1 -> output:#18#28
- U$242: device output:#A1#1 -> SparkFun-Aesthetics:SFE_LOGO_FLAME_.1
- U$243: device output:#A2#4 -> output:#LD#29
- U$244: device output:#0#4 -> output:1830
- U$245: device output:#1#4 -> output:RGB_14141832
- U$246: device output:#2#CS#5 -> output:#VB26
- U$247: device output:#3#SCK#5 -> output:CUR1714141837
- U$248: device output:#4#PICO#5 -> output:#MEAS#1714141838
- U$249: device output:#5#POCI#5 -> output:THING_PLUS1714141839
- U$25: device output:16165 -> output:THING_PLUS1714141839
- U$250: device output:#6#RX1#6 -> output:NORA#W3061714141840
- U$251: device output:#7#TX1#7 -> output:#GND#ON#3061714141842
- U$252: device output:#8#8 -> output:23061714141843
- U$253: device output:#SDA#9#10 -> output:#17#11
- U$254: device output:#SCL#10#10 -> output:SDPC23061714141844
- U$255: device output:#11#11 -> output:##RST##23061714141845
- U$256: device output:#12#12 -> output:#JP3#23061714141846
- U$257: device output:#13#13 -> output:#100#23061714141846
- U$258: device output:#14#14 -> output:#500#23061714141846
- U$26: device output:#SDA#9#10 -> output:#VB26
- U$27: device output:#SCL#10#10 -> output:CUR1714141837
- U$28: device output:#11#11 -> output:NORA#W3061714141840
- U$29: device output:#12#12 -> output:23061714141843
- U$3: device output:CHG0 -> output:#MEAS#1714141838
- U$34: device output:1417 -> output:SDPC23061714141844
- U$35: device output:#10#91420 -> output:#18#18
- U$4: device output:#100#501 -> output:CHG0
- U$42: device output:#VBAT#0 -> output:#JP3#23061714141846
- U$57: device output:#G#18 -> output:#3V#23
- U$58: device output:#JP3#0 -> output:#JP2#0
- U$59: device output:CHG0 -> output:#VUSB#0
- U$6: device output:NORA#W3060 -> output:##RST##23061714141845
- U$61: device output:##RESET##0 -> output:#100#23061714141846
- U$65: device output:#NC#1 -> output:#JP1#0
- U$70: device output:#JP1#18 -> output:#9#10
- U$71: device output:#JP2#18 -> output:#LED_DO#0
- U$73: device output:RGB_155 -> output:#500#23061714141846
- U$74: device output:#JP4#0 -> output:#10#11
- U$75: device output:RESET0 -> output:#G#22
- U$76: device output:#VUSB#0 -> output:#VU#23
- U$77: device output:#VBAT#0 -> output:#VB26
- U$8: device SparkFun-Aesthetics:SFE_LOGO_FLAME_.1 -> SparkFun-Aesthetics:SFE_LOGO_FLAME_.2
- U$80: device output:#EN#0 -> output:#EN#27
- U$81: device output:#3V3#0 -> output:#2#28
- U$82: device output:CHG0 -> output:#3#28
- U$83: device output:MA0 -> output:#4#CS#28
- U$84: device output:THING_PLUS_0 -> output:#5#SCK#28
- U$85: device output:BOOT0 -> output:#6#PICO#28
- U$87: device output:PWR0 -> output:#9#TX1#A2#28
- U$88: device output:NORA#W3060 -> output:#8#RX1#A1#28
- U$89: device output:NORA#W3060 -> output:#EN#0
- U$9: device output:#500#501 -> output:RESET0
- U$90: device SparkFun-Aesthetics:SFE_LOGO_FLAME_.1 -> output:#3V3#0
- U$91: device output:#A0#1 -> output:#10#28
- U$92: device output:#A1#1 -> output:MA0
- U$93: device output:#A2#4 -> output:THING_PLUS_0
- U$94: device output:#0#4 -> output:BOOT0
- U$95: device output:#1#4 -> output:PWR0
- U$96: device output:#2#CS#5 -> output:NORA#W3060
- U$97: device output:#3#SCK#5 -> SparkFun-Aesthetics:SFE_LOGO_FLAME_.2
- U$98: device output:#4#PICO#5 -> output:#A0#1
- U$99: device output:#5#POCI#5 -> output:#0#4
- U10, U15, U6: value CP2102N_QFN28 -> CP2102N; device nora-w306:QFN28 -> SparkFun-IC-Comms:QFN24
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Connections:
- removed net !RESET!3: C52.1, J22.28, J24.10, Q8.3, S10.1, S10.2, U18.J3
- removed net !RESET!4: C65.1, J28.28, J30.10, Q10.3, S13.1, S13.2, U23.J3
- removed net !RESET!5: C78.1, J34.28, J36.10, Q12.3, S16.1, S16.2, U28.J3
- removed net !RESET!6: C91.1, J40.28, J42.10, Q14.3, S19.1, S19.2, U33.J3
- removed net !RESET!7: C104.1, J46.28, J48.10, Q16.3, S22.1, S22.2, U38.J3
- removed net !RESET!8: C117.1, J52.28, J54.10, Q18.3, S25.1, S25.2, U43.J3
- removed net !RESET!9: C130.1, J58.28, J60.10, Q20.3, S28.1, S28.2, U48.J3
- removed net 3.3V3: C41.1, C44.1, C45.1, C46.1, C47.1, C48.1, C49.1, C51.1, D24.VCC, E4.2, E4.5, I2C3.2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
- removed net 3.3V4: C54.1, C57.1, C58.1, C59.1, C60.1, C61.1, C62.1, C64.1, D30.VCC, E5.2, E5.5, I2C4.2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
- removed net 3.3V5: C67.1, C70.1, C71.1, C72.1, C73.1, C74.1, C75.1, C77.1, D36.VCC, E6.2, E6.5, I2C5.2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
- removed net 3.3V6: C80.1, C83.1, C84.1, C85.1, C86.1, C87.1, C88.1, C90.1, D42.VCC, E7.2, E7.5, I2C6.2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
- removed net 3.3V7: C100.1, C101.1, C103.1, C93.1, C96.1, C97.1, C98.1, C99.1, D48.VCC, E8.2, E8.5, I2C7.2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
- removed net 3.3V8: C106.1, C109.1, C110.1, C111.1, C112.1, C113.1, C114.1, C116.1, D54.VCC, E9.2, E9.5, I2C8.2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
- removed net 3.3V9: C119.1, C122.1, C123.1, C124.1, C125.1, C126.1, C127.1, C129.1, D60.VCC, E10.2, E10.5, I2C9.2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
- removed net CC10: J27.A5, R82.2
- removed net CC11: J33.B5, R99.2
- removed net CC12: J33.A5, R100.2
- removed net CC13: J39.B5, R117.2
- removed net CC14: J39.A5, R118.2
- removed net CC15: J45.B5, R135.2
- removed net CC16: J45.A5, R136.2
- removed net CC17: J51.B5, R153.2
- removed net CC18: J51.A5, R154.2
- removed net CC19: J57.B5, R171.2
- removed net CC20: J57.A5, R172.2
- removed net CC7: J21.B5, R63.2
- removed net CC8: J21.A5, R64.2
- removed net CC9: J27.B5, R81.2
- removed net CHG3: CHG3.2, U16.1
- removed net CHG4: CHG4.2, U21.1
- removed net CHG5: CHG5.2, U26.1
- removed net CHG6: CHG6.2, U31.1
- removed net CHG7: CHG7.2, U36.1
- removed net CHG8: CHG8.2, U41.1
- removed net CHG9: CHG9.2, U46.1
- removed net DTR3: Q8.1, R68.1, U20.28
- removed net DTR4: Q10.1, R86.1, U25.28
- removed net DTR5: Q12.1, R104.1, U30.28
- removed net DTR6: Q14.1, R122.1, U35.28
- removed net DTR7: Q16.1, R140.1, U40.28
- removed net DTR8: Q18.1, R158.1, U45.28
- removed net DTR9: Q20.1, R176.1, U50.28
- removed net EN3: J22.11, R60.2, U17.3
- removed net EN4: J28.11, R78.2, U22.3
- removed net EN5: J34.11, R96.2, U27.3
- removed net EN6: J40.11, R114.2, U32.3
- removed net EN7: J46.11, R132.2, U37.3
- removed net EN8: J52.11, R150.2, U42.3
- removed net EN9: J58.11, R168.2, U47.3
- removed net GND3: C40.2, C41.2, C42.2, C43.2, C44.2, C45.2, C46.2, C47.2, C48.2, C49.2, C50.2, C51.2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
- removed net GND4: C53.2, C54.2, C55.2, C56.2, C57.2, C58.2, C59.2, C60.2, C61.2, C62.2, C63.2, C64.2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
- removed net GND5: C66.2, C67.2, C68.2, C69.2, C70.2, C71.2, C72.2, C73.2, C74.2, C75.2, C76.2, C77.2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
- removed net GND6: C79.2, C80.2, C81.2, C82.2, C83.2, C84.2, C85.2, C86.2, C87.2, C88.2, C89.2, C90.2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
- removed net GND7: C100.2, C101.2, C102.2, C103.2, C104.2, C92.2, C93.2, C94.2, C95.2, C96.2, C97.2, C98.2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
- removed net GND8: C105.2, C106.2, C107.2, C108.2, C109.2, C110.2, C111.2, C112.2, C113.2, C114.2, C115.2, C116.2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
- removed net GND9: C118.2, C119.2, C120.2, C121.2, C122.2, C123.2, C124.2, C125.2, C126.2, C127.2, C128.2, C129.2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
- removed net N$100: JP16.2, R59.1
- removed net N$101: D26.A, R74.2
- removed net N$102: R76.2, U25.9
- removed net N$103: D27.A, R77.2
- removed net N$104: R79.1, R80.2, U25.8
- removed net N$105: CUR4.2, U21.5
- removed net N$106: CUR4.1, R83.1
- removed net N$107: CUR4.3, R75.2
- removed net N$108: Q9.1, R84.2
- removed net N$109: R85.2, S14.3, S14.4
- removed net N$110: Q10.5, R86.2
- removed net N$111: Q10.2, R87.2
- removed net N$112: LED4.2, R88.1
- removed net N$113: D28.A, R88.2
- removed net N$114: D29.6, U25.4
- removed net N$115: D29.1, J27.A6, J27.B6
- removed net N$116: D29.4, U25.5
- removed net N$117: D29.3, J27.A7, J27.B7
- removed net N$118: D30.DO, TP5.1
- removed net N$119: E5.1, JP18.1
- removed net N$120: E5.4, JP17.1
- removed net N$121: CHG4.1, D26.C
- removed net N$122: D30.DI, JP19.2
- removed net N$123: I2C4.3, R89.2
- removed net N$124: I2C4.1, R90.2
- removed net N$125: JP20.2, R77.1
- removed net N$126: D32.A, R92.2
- removed net N$127: R94.2, U30.9
- removed net N$128: D33.A, R95.2
- removed net N$129: R97.1, R98.2, U30.8
- removed net N$130: CUR5.2, U26.5
- removed net N$131: CUR5.1, R101.1
- removed net N$132: CUR5.3, R93.2
- removed net N$133: Q11.1, R102.2
- removed net N$134: R103.2, S17.3, S17.4
- removed net N$135: Q12.5, R104.2
- removed net N$136: Q12.2, R105.2
- removed net N$137: LED5.2, R106.1
- removed net N$138: D34.A, R106.2
- removed net N$139: D35.6, U30.4
- removed net N$140: D35.1, J33.A6, J33.B6
- removed net N$141: D35.4, U30.5
- removed net N$142: D35.3, J33.A7, J33.B7
- removed net N$143: D36.DO, TP6.1
- removed net N$144: E6.1, JP22.1
- removed net N$145: E6.4, JP21.1
- removed net N$146: CHG5.1, D32.C
- removed net N$147: D36.DI, JP23.2
- removed net N$148: I2C5.3, R107.2
- removed net N$149: I2C5.1, R108.2
- removed net N$150: JP24.2, R95.1
- removed net N$151: D38.A, R110.2
- removed net N$152: R112.2, U35.9
- removed net N$153: D39.A, R113.2
- removed net N$154: R115.1, R116.2, U35.8
- removed net N$155: CUR6.2, U31.5
- removed net N$156: CUR6.1, R119.1
- removed net N$157: CUR6.3, R111.2
- removed net N$158: Q13.1, R120.2
- removed net N$159: R121.2, S20.3, S20.4
- removed net N$160: Q14.5, R122.2
- removed net N$161: Q14.2, R123.2
- removed net N$162: LED6.2, R124.1
- removed net N$163: D40.A, R124.2
- removed net N$164: D41.6, U35.4
- removed net N$165: D41.1, J39.A6, J39.B6
- removed net N$166: D41.4, U35.5
- removed net N$167: D41.3, J39.A7, J39.B7
- removed net N$168: D42.DO, TP7.1
- removed net N$169: E7.1, JP26.1
- removed net N$170: E7.4, JP25.1
- removed net N$171: CHG6.1, D38.C
- removed net N$172: D42.DI, JP27.2
- removed net N$173: I2C6.3, R125.2
- removed net N$174: I2C6.1, R126.2
- removed net N$175: JP28.2, R113.1
- removed net N$176: D44.A, R128.2
- removed net N$177: R130.2, U40.9
- removed net N$178: D45.A, R131.2
- removed net N$179: R133.1, R134.2, U40.8
- removed net N$180: CUR7.2, U36.5
- removed net N$181: CUR7.1, R137.1
- removed net N$182: CUR7.3, R129.2
- removed net N$183: Q15.1, R138.2
- removed net N$184: R139.2, S23.3, S23.4
- removed net N$185: Q16.5, R140.2
- removed net N$186: Q16.2, R141.2
- removed net N$187: LED7.2, R142.1
- removed net N$188: D46.A, R142.2
- removed net N$189: D47.6, U40.4
- removed net N$190: D47.1, J45.A6, J45.B6
- removed net N$191: D47.4, U40.5
- removed net N$192: D47.3, J45.A7, J45.B7
- removed net N$193: D48.DO, TP8.1
- removed net N$194: E8.1, JP30.1
- removed net N$195: E8.4, JP29.1
- removed net N$196: CHG7.1, D44.C
- removed net N$197: D48.DI, JP31.2
- removed net N$198: I2C7.3, R143.2
- removed net N$199: I2C7.1, R144.2
- removed net N$200: JP32.2, R131.1
- removed net N$201: D50.A, R146.2
- removed net N$202: R148.2, U45.9
- removed net N$203: D51.A, R149.2
- removed net N$204: R151.1, R152.2, U45.8
- removed net N$205: CUR8.2, U41.5
- removed net N$206: CUR8.1, R155.1
- removed net N$207: CUR8.3, R147.2
- removed net N$208: Q17.1, R156.2
- removed net N$209: R157.2, S26.3, S26.4
- removed net N$210: Q18.5, R158.2
- removed net N$211: Q18.2, R159.2
- removed net N$212: LED8.2, R160.1
- removed net N$213: D52.A, R160.2
- removed net N$214: D53.6, U45.4
- removed net N$215: D53.1, J51.A6, J51.B6
- removed net N$216: D53.4, U45.5
- removed net N$217: D53.3, J51.A7, J51.B7
- removed net N$218: D54.DO, TP9.1
- removed net N$219: E9.1, JP34.1
- removed net N$220: E9.4, JP33.1
- removed net N$221: CHG8.1, D50.C
- removed net N$222: D54.DI, JP35.2
- removed net N$223: I2C8.3, R161.2
- removed net N$224: I2C8.1, R162.2
- removed net N$225: JP36.2, R149.1
- removed net N$226: D56.A, R164.2
- removed net N$227: R166.2, U50.9
- removed net N$228: D57.A, R167.2
- removed net N$229: R169.1, R170.2, U50.8
- removed net N$230: CUR9.2, U46.5
- removed net N$231: CUR9.1, R173.1
- removed net N$232: CUR9.3, R165.2
- removed net N$233: Q19.1, R174.2
- removed net N$234: R175.2, S29.3, S29.4
- removed net N$235: Q20.5, R176.2
- removed net N$236: Q20.2, R177.2
- removed net N$237: LED9.2, R178.1
- removed net N$238: D58.A, R178.2
- removed net N$239: D59.6, U50.4
- removed net N$240: D59.1, J57.A6, J57.B6
- removed net N$241: D59.4, U50.5
- removed net N$242: D59.3, J57.A7, J57.B7
- removed net N$243: D60.DO, TP10.1
- removed net N$244: E10.1, JP38.1
- removed net N$245: E10.4, JP37.1
- removed net N$246: CHG9.1, D56.C
- removed net N$247: D60.DI, JP39.2
- removed net N$248: I2C9.3, R179.2
- removed net N$249: I2C9.1, R180.2
- removed net N$250: JP40.2, R167.1
- removed net N$37 (its old number): LED1.2, R34.1
- removed net N$47 (its old number): D12.DI, JP7.2
- removed net N$49 (its old number): I2C1.1, R36.2
- removed net N$50 (its old number): JP8.2, R21.1
- removed net N$69 (its old number): E3.1, JP10.1
- removed net N$79 (its old number): R61.1, R62.2, U20.8
- removed net N$81 (its old number): CUR3.1, R65.1
- removed net N$82 (its old number): CUR3.3, R57.2
- removed net N$97: D24.DI, JP15.2
- removed net N$98: I2C3.3, R71.2
- removed net N$99: I2C3.1, R72.2
- removed net PA12/PICO: J1.17, J4.3, U1.J9
- removed net PA12/PICO1: J10.17, J11.3, U8.J9
- removed net PA12/PICO2: J16.17, J17.3, U13.J9
- removed net PA12/PICO3: J22.17, J23.3, U18.J9
- removed net PA12/PICO4: J28.17, J29.3, U23.J9
- removed net PA12/PICO5: J34.17, J35.3, U28.J9
- removed net PA12/PICO6: J40.17, J41.3, U33.J9
- removed net PA12/PICO7: J46.17, J47.3, U38.J9
- removed net PA12/PICO8: J52.17, J53.3, U43.J9
- removed net PA12/PICO9: J58.17, J59.3, U48.J9
- removed net PA13/POCI: J1.16, J4.7, U1.J8
- removed net PA13/POCI1: J10.16, J11.7, U8.J8
- removed net PA13/POCI2: J16.16, J17.7, U13.J8
- removed net PA13/POCI3: J22.16, J23.7, U18.J8
- removed net PA13/POCI4: J28.16, J29.7, U23.J8
- removed net PA13/POCI5: J34.16, J35.7, U28.J8
- removed net PA13/POCI6: J40.16, J41.7, U33.J8
- removed net PA13/POCI7: J46.16, J47.7, U38.J8
- removed net PA13/POCI8: J52.16, J53.7, U43.J8
- removed net PA13/POCI9: J58.16, J59.7, U48.J8
- removed net PA14/SCK: J1.18, J4.5, U1.H9
- removed net PA14/SCK1: J10.18, J11.5, U8.H9
- removed net PA14/SCK2: J16.18, J17.5, U13.H9
- removed net PA14/SCK3: J22.18, J23.5, U18.H9
- removed net PA14/SCK4: J28.18, J29.5, U23.H9
- removed net PA14/SCK5: J34.18, J35.5, U28.H9
- removed net PA14/SCK6: J40.18, J41.5, U33.H9
- removed net PA14/SCK7: J46.18, J47.5, U38.H9
- removed net PA14/SCK8: J52.18, J53.5, U43.H9
- removed net PA14/SCK9: J58.18, J59.5, U48.H9
- removed net PA15/CS: J1.19, J4.2, U1.H8
- removed net PA15/CS1: J10.19, J11.2, U8.H8
- removed net PA15/CS2: J16.19, J17.2, U13.H8
- removed net PA15/CS3: J22.19, J23.2, U18.H8
- removed net PA15/CS4: J28.19, J29.2, U23.H8
- removed net PA15/CS5: J34.19, J35.2, U28.H8
- removed net PA15/CS6: J40.19, J41.2, U33.H8
- removed net PA15/CS7: J46.19, J47.2, U38.H8
- removed net PA15/CS8: J52.19, J53.2, U43.H8
- removed net PA15/CS9: J58.19, J59.2, U48.H8
- removed net PA17: J40.3, U33.B1
- removed net PA18: J40.4, U33.B3
- removed net PA19: J46.13, U38.H2
- removed net PA20: J46.3, U38.B1
- removed net PA21: J46.4, U38.B3
- removed net PA22: J52.13, U43.H2
- removed net PA23: J52.3, U43.B1
- removed net PA24: J52.4, U43.B3
- removed net PA25: J58.13, U48.H2
- removed net PA25/LP_UART_RXD: J1.15, U1.C2
- removed net PA25/LP_UART_RXD1: J10.15, U8.C2
- removed net PA25/LP_UART_RXD2: J16.15, U13.C2
- removed net PA25/LP_UART_RXD3: J22.15, U18.C2
- removed net PA25/LP_UART_RXD4: J28.15, U23.C2
- removed net PA25/LP_UART_RXD5: J34.15, U28.C2
- removed net PA25/LP_UART_RXD6: J40.15, U33.C2
- removed net PA25/LP_UART_RXD7: J46.15, U38.C2
- removed net PA25/LP_UART_RXD8: J52.15, U43.C2
- removed net PA25/LP_UART_RXD9: J58.15, U48.C2
- removed net PA26: J58.3, U48.B1
- removed net PA26/LP_UART_TXD: J1.14, U1.C1
- removed net PA26/LP_UART_TXD1: J10.14, U8.C1
- removed net PA26/LP_UART_TXD2: J16.14, U13.C1
- removed net PA26/LP_UART_TXD3: J22.14, U18.C1
- removed net PA26/LP_UART_TXD4: J28.14, U23.C1
- removed net PA26/LP_UART_TXD5: J34.14, U28.C1
- removed net PA26/LP_UART_TXD6: J40.14, U33.C1
- removed net PA26/LP_UART_TXD7: J46.14, U38.C1
- removed net PA26/LP_UART_TXD8: J52.14, U43.C1
- removed net PA26/LP_UART_TXD9: J58.14, U48.C1
- removed net PA27: J1.13, U1.H2
- removed net PA29: J58.4, U48.B3
- removed net PA7/UART-LOG-TXD3: J22.20, Q8.6, S11.1, S11.2, U18.A5, U20.25
- removed net PA7/UART-LOG-TXD4: J28.20, Q10.6, S14.1, S14.2, U23.A5, U25.25
- removed net PA7/UART-LOG-TXD5: J34.20, Q12.6, S17.1, S17.2, U28.A5, U30.25
- removed net PA7/UART-LOG-TXD6: J40.20, Q14.6, S20.1, S20.2, U33.A5, U35.25
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Routing:
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- removed copper zone on layer 1, net 3.3V3
- removed copper zone on layer 15, net 3.3V3
- removed copper zone on layer 1, net 3.3V4
- removed copper zone on layer 15, net 3.3V4
- removed copper zone on layer 1, net 3.3V5
- removed copper zone on layer 15, net 3.3V5
- removed copper zone on layer 1, net 3.3V6
- removed copper zone on layer 15, net 3.3V6
- removed copper zone on layer 1, net 3.3V7
- removed copper zone on layer 15, net 3.3V7
- removed copper zone on layer 1, net 3.3V8
- removed copper zone on layer 15, net 3.3V8
- removed copper zone on layer 1, net 3.3V9
- removed copper zone on layer 15, net 3.3V9
- removed copper zone on layer 1, net GND3
- removed copper zone on layer 16, net GND3
- removed copper zone on layer 2, net GND3
- removed copper zone on layer 1, net GND4
- removed copper zone on layer 16, net GND4
- removed copper zone on layer 2, net GND4
- removed copper zone on layer 1, net GND5
- removed copper zone on layer 16, net GND5
- removed copper zone on layer 2, net GND5
- removed copper zone on layer 1, net GND6
- removed copper zone on layer 16, net GND6
- removed copper zone on layer 2, net GND6
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Other:
- board size 130 x 141.7 mm -> 83.3 x 80.3 mm
- board text added: "v04"
- board text removed: "v03"
