File: Hardware/Production/SparkFun_Thing_Plus_NORA_W306-Panel.brd (EAGLE design)
At the start: 83.3 x 80.3 mm, 513 parts, among them J1 THING_PLUS_LOGICAL, J10 THING_PLUS_LOGICAL, J11 SDFRICTION, J12 SWD (DNP), J13 LiPo, J14 QWIIC_RA, J15 USB-C, J16 THING_PLUS_LOGICAL, J17 SDFRICTION, J18 SWD (DNP), J2 LiPo, J3 QWIIC_RA, J4 SDFRICTION, J5 USB-C, J6 SWD (DNP), J7 LiPo, J8 QWIIC_RA, J9 USB-C, Q1 20V/4.2A/52mΩ/1.4W, Q10 20V/0.2A/8MHz/1.2Ω/1Vth, Q11 20V/4.2A/52mΩ/1.4W, Q12 MBT3904DW1T1, Q13 20V/4.2A/52mΩ/1.4W, Q14 20V/4.2A/52mΩ/1.4W, Q15 20V/0.2A/8MHz/1.2Ω/1Vth, Q2 MBT3904DW1T1, Q3 20V/4.2A/52mΩ/1.4W, Q4 20V/4.2A/52mΩ/1.4W, Q5 20V/0.2A/8MHz/1.2Ω/1Vth, Q6 20V/4.2A/52mΩ/1.4W, Q7 MBT3904DW1T1, Q8 20V/4.2A/52mΩ/1.4W, Q9 20V/4.2A/52mΩ/1.4W, U1 UBLOX_NORA_W306, U10 CP2102N, U11 MCP73831, U12 XC6222B331MR-G, U13 UBLOX_NORA_W306, U14 MAX17048, U15 CP2102N, U2 MCP73831, U3 XC6222B331MR-G, U4 MCP73831, U5 MAX17048, U6 CP2102N, U7 XC6222B331MR-G, U8 UBLOX_NORA_W306, U9 MAX17048

Commit message: Production panel and gerbers v10
Parts:
- added C100, C103, C111, C112, C115, C123, C124, C127, C135, C136, C139, C39, C40, C43, C51, C52, C55, C63, C64, C67, C75, C76, C79, C87, C88, C91, C99: 4.7uF, SparkFun-Capacitors:0603
- added C101, C104, C105, C113, C116, C117, C125, C128, C129, C137, C140, C141, C41, C44, C45, C53, C56, C57, C65, C68, C69, C77, C80, C81, C89, C92, C93: 10uF, SparkFun-Capacitors:0402-TIGHT
- added C102, C106, C107, C108, C114, C118, C119, C120, C126, C130, C131, C132, C138, C142, C143, C144, C42, C46, C47, C48, C54, C58, C59, C60, C66, C70, C71, C72, C78, C82, C83, C84, C90, C94, C95, C96: 0.1uF, SparkFun-Capacitors:0402-TIGHT
- added C109, C110, C121, C122, C133, C134, C37, C38, C49, C50, C61, C62, C73, C74, C85, C86, C97, C98: 1.0uF, SparkFun-Capacitors:0402-TIGHT
- added CHG10, CHG11, CHG3, CHG4, CHG5, CHG6, CHG7, CHG8, CHG9, JP10, JP11, JP12, JP13, JP14, JP15, JP16, JP17, JP18, JP19, JP20, JP21, JP22, JP23, JP24, JP25, JP26, JP27, JP28, JP29, JP30, JP31, JP32, JP33, JP34, JP35, JP36, LED10, LED11, LED3, LED4, LED5, LED6, LED7, LED8, LED9, USBSHLD10, USBSHLD11, USBSHLD3, USBSHLD4, USBSHLD5, USBSHLD6, USBSHLD7, USBSHLD8, USBSHLD9: (no value), SparkFun-Jumpers:SMT-JUMPER_2_NC_TRACE_SILK
- added CUR10, CUR11, CUR3, CUR4, CUR5, CUR6, CUR7, CUR8, CUR9, SDPC10, SDPC11, SDPC3, SDPC4, SDPC5, SDPC6, SDPC7, SDPC8, SDPC9: (no value), SparkFun-Jumpers:SMT-JUMPER_3_1-NC_TRACE_SILK
- added D19, D25, D31, D37, D43, D49, D55, D61, D67: 1A/23V/620mV, SparkFun-DiscreteSemi:SOD-323
- added D20, D26, D32, D38, D44, D50, D56, D62, D68: Yellow, SparkFun-LED:LED-0603
- added D21, D27, D33, D39, D45, D51, D57, D63, D69: BLUE, SparkFun-LED:LED-0603
- added D22, D28, D34, D40, D46, D52, D58, D64, D70: RED, SparkFun-LED:LED-0603
- added D23, D29, D35, D41, D47, D53, D59, D65, D71: PRTR5V0U2F, SparkFun-IC-Power:SOT886
- added D24, D30, D36, D42, D48, D54, D60, D66, D72: WS2812, SparkFun-LED:WS2812-2020
- added FD13, FD14, FD15, FD16, FD17, FD18, FD19, FD20, FD21, FD22, FD23, FD24, FD25, FD26, FD27, FD28, FD29, FD30, FD31, FD32, FD33, FD34, FD35, FD36, FD37, FD38, FD39, FD40, FD41, FD42, FD43, FD44, FD45, FD46, FD47, FD48: FIDUCIALUFIDUCIAL, SparkFun-Aesthetics:FIDUCIAL-MICRO
- added H13, H14, H15, H16, H17, H18, H19, H20, H21, H22, H23, H24, H25, H26, H27, H28, H29, H30, H31, H32, H33, H34, H35, H36, H37, H38, H39, H40, H41, H42, H43, H44, H45, H46, H47, H48: STAND-OFF, SparkFun-Hardware:STAND-OFF
- added I2C10, I2C11, I2C3, I2C4, I2C5, I2C6, I2C7, I2C8, I2C9: JUMPER-SMT_3_2-NC_TRACE_SILK, SparkFun-Jumpers:SMT-JUMPER_3_2-NC_TRACE_SILK
- added J19, J25, J31, J37, J43, J49, J55, J61, J67: LiPo, SparkFun-Connectors:JST-2-SMD
- added J20, J26, J32, J38, J44, J50, J56, J62, J68: QWIIC_RIGHT_ANGLE, SparkFun-Connectors:JST04_1MM_RA
- added J21, J27, J33, J39, J45, J51, J57, J63, J69: USB-C, SparkFun-Connectors:USB-C-16P-4LAYER-ISOLATED
- added J22, J28, J34, J40, J46, J52, J58, J64, J70: THING_PLUS_LOGICAL, SparkFun-Boards:THING_PLUS
- added J23, J29, J35, J41, J47, J53, J59, J65, J71: SDFRICTION, SparkFun-Connectors:MICROSD_TINY
- added J24, J30, J36, J42, J48, J54, J60, J66, J72: SWD (DNP), SparkFun-Connectors:2X5-SMD-UNSHROUDED_DNP_NO_PASTE
- added LOGO10, LOGO13, LOGO16, LOGO19, LOGO22, LOGO25, LOGO28, LOGO31, LOGO34: OSHW-LOGOM, SparkFun-Aesthetics:OSHW-LOGO-M
- added LOGO11, LOGO14, LOGO17, LOGO20, LOGO23, LOGO26, LOGO29, LOGO32, LOGO35: QWIIC_LOGO_4MM, SparkFun-Aesthetics:QWIIC_4MM
- added LOGO12, LOGO15, LOGO18, LOGO21, LOGO24, LOGO27, LOGO30, LOGO33, LOGO36: SFE_LOGO_NAME_FLAME.1_INCH, SparkFun-Aesthetics:SFE_LOGO_NAME_FLAME_.1
- added MEAS10, MEAS11, MEAS3, MEAS4, MEAS5, MEAS6, MEAS7, MEAS8, MEAS9: (no value), SparkFun-Jumpers:COMBO-JUMPER_2_NC_TRACE
- added Q16, Q18, Q19, Q21, Q23, Q24, Q26, Q28, Q29, Q31, Q33, Q34, Q36, Q38, Q39, Q41, Q43, Q44, Q46, Q48, Q49, Q51, Q53, Q54, Q56, Q58, Q59: 20V/4.2A/52mΩ/1.4W, SparkFun-DiscreteSemi:SOT23-3
- added Q17, Q22, Q27, Q32, Q37, Q42, Q47, Q52, Q57: MBT3904DW1T1, SparkFun-DiscreteSemi:SC70-6
- added Q20, Q25, Q30, Q35, Q40, Q45, Q50, Q55, Q60: 20V/0.2A/8MHz/1.2Ω/1Vth, SparkFun-DiscreteSemi:SOT-416FL
- added R100, R112, R119, R123, R125, R137, R144, R148, R150, R162, R169, R173, R175, R187, R194, R198, R200, R212, R219, R223, R225, R237, R244, R248, R250, R262, R269, R273, R275, R287, R294, R298, R300, R87, R94, R98: 100, SparkFun-Resistors:0402-TIGHT
- added R101, R106, R120, R121, R122, R126, R131, R145, R146, R147, R151, R156, R170, R171, R172, R176, R181, R195, R196, R197, R201, R206, R220, R221, R222, R226, R231, R245, R246, R247, R251, R256, R270, R271, R272, R276, R281, R295, R296, R297, R76, R81, R95, R96, R97: 100k, SparkFun-Resistors:0402-TIGHT
- added R102, R105, R116, R127, R130, R141, R152, R155, R166, R177, R180, R191, R202, R205, R216, R227, R230, R241, R252, R255, R266, R277, R280, R291, R77, R80, R91: 4.7k, SparkFun-Resistors:0402-TIGHT
- added R103, R128, R153, R178, R203, R228, R253, R278, R78: 2.0k, SparkFun-Resistors:0603
- added R104, R111, R114, R115, R129, R136, R139, R140, R154, R161, R164, R165, R179, R186, R189, R190, R204, R211, R214, R215, R229, R236, R239, R240, R254, R261, R264, R265, R279, R286, R289, R290, R79, R86, R89, R90: 10k, SparkFun-Resistors:0402-TIGHT
- added R107, R132, R157, R182, R207, R232, R257, R282, R82: 22k, SparkFun-Resistors:0402-TIGHT
- added R108, R133, R158, R183, R208, R233, R258, R283, R83: 33k, SparkFun-Resistors:0402-TIGHT
- added R109, R110, R134, R135, R159, R160, R184, R185, R209, R210, R234, R235, R259, R260, R284, R285, R84, R85: 5.1k, SparkFun-Resistors:0402-TIGHT
- added R113, R124, R138, R149, R163, R174, R188, R199, R213, R224, R238, R249, R263, R274, R288, R299, R88, R99: 1k, SparkFun-Resistors:0402-TIGHT
- added R117, R118, R142, R143, R167, R168, R192, R193, R217, R218, R242, R243, R267, R268, R292, R293, R92, R93: 2.2k, SparkFun-Resistors:0402-TIGHT
- added S10, S13, S16, S19, S22, S25, S28, S31, S34: RESET, SparkFun-Switches:TACTILE_SWITCH_SMD_4.6X2.8MM
- added S11, S14, S17, S20, S23, S26, S29, S32, S35: BOOT, SparkFun-Switches:TACTILE_SWITCH_SMD_4.6X2.8MM
- added S12, S15, S18, S21, S24, S27, S30, S33, S36: USER, SparkFun-Switches:TACTILE_SWITCH_SMD_4.6X2.8MM
- added U$1000, U$320, U$405, U$490, U$575, U$660, U$745, U$830, U$915: (no value), output:#SDA#11#28
- added U$1001, U$321, U$406, U$491, U$576, U$661, U$746, U$831, U$916: (no value), output:#SCL#12#28
- added U$1002, U$322, U$407, U$492, U$577, U$662, U$747, U$832, U$917: (no value), output:#17#28
- added U$1003, U$323, U$408, U$493, U$578, U$663, U$748, U$833, U$918: (no value), output:#18#28
- added U$1004, U$324, U$409, U$494, U$579, U$664, U$749, U$834, U$919: (no value), SparkFun-Aesthetics:SFE_LOGO_FLAME_.1
- added U$1005, U$325, U$410, U$495, U$580, U$665, U$750, U$835, U$920: (no value), output:#LD#29
- added U$1006, U$309, U$326, U$394, U$411, U$479, U$496, U$564, U$581, U$649, U$666, U$734, U$751, U$819, U$836, U$904, U$921, U$989: (no value), output:#VB26
- added U$1007, U$327, U$412, U$497, U$582, U$667, U$752, U$837, U$922: (no value), output:#MEAS#1714141838
- added U$1008, U$328, U$413, U$498, U$583, U$668, U$753, U$838, U$923: (no value), output:THING_PLUS1714141839
- added U$1009, U$329, U$414, U$499, U$584, U$669, U$754, U$839, U$924: (no value), output:NORA#W3061714141840
- added U$1010, U$330, U$415, U$500, U$585, U$670, U$755, U$840, U$925: (no value), output:#GND#ON#3061714141842
- added U$1011, U$302, U$331, U$387, U$416, U$472, U$501, U$557, U$586, U$642, U$671, U$727, U$756, U$812, U$841, U$897, U$926, U$982: (no value), output:#17#11
- added U$1012, U$332, U$417, U$502, U$587, U$672, U$757, U$842, U$927: (no value), output:##RST##23061714141845
- added U$1013, U$333, U$418, U$503, U$588, U$673, U$758, U$843, U$928: (no value), output:#JP3#23061714141846
- added U$1014, U$334, U$419, U$504, U$589, U$674, U$759, U$844, U$929: (no value), output:#100#23061714141846
- added U$1015, U$335, U$420, U$505, U$590, U$675, U$760, U$845, U$930: (no value), output:#500#23061714141846
- added U$1016, U$336, U$421, U$506, U$591, U$676, U$761, U$846, U$931: (no value), output:IO180
- added U$1017, U$337, U$422, U$507, U$592, U$677, U$762, U$847, U$932: (no value), output:IO20
- added U$1018, U$338, U$423, U$508, U$593, U$678, U$763, U$848, U$933: (no value), output:RGB_IO140
- added U$1019, U$339, U$424, U$509, U$594, U$679, U$764, U$849, U$934: (no value), output:#CUR#0
- added U$1020, U$340, U$425, U$510, U$595, U$680, U$765, U$850, U$935: (no value), output:#SDPC#0
- added U$259, U$344, U$429, U$514, U$599, U$684, U$769, U$854, U$939: (no value), output:#EN#0
- added U$260, U$345, U$430, U$515, U$600, U$685, U$770, U$855, U$940: (no value), output:#3V3#0
- added U$261, U$346, U$431, U$516, U$601, U$686, U$771, U$856, U$941: (no value), output:THING_PLUS_0
- added U$262, U$347, U$432, U$517, U$602, U$687, U$772, U$857, U$942: (no value), output:BOOT0
- added U$263, U$348, U$433, U$518, U$603, U$688, U$773, U$858, U$943: (no value), output:PWR0
- added U$264, U$349, U$434, U$519, U$604, U$689, U$774, U$859, U$944: (no value), output:NORA#W3060
- added U$265, U$350, U$435, U$520, U$605, U$690, U$775, U$860, U$945: (no value), SparkFun-Aesthetics:SFE_LOGO_FLAME_.2
- added U$266, U$351, U$436, U$521, U$606, U$691, U$776, U$861, U$946: (no value), output:#A0#1
- added U$267, U$352, U$437, U$522, U$607, U$692, U$777, U$862, U$947: (no value), output:#0#4
- added U$268, U$353, U$438, U$523, U$608, U$693, U$778, U$863, U$948: (no value), output:#1#4
- added U$269, U$354, U$439, U$524, U$609, U$694, U$779, U$864, U$949: (no value), output:#13#13
- added U$270, U$355, U$440, U$525, U$610, U$695, U$780, U$865, U$950: (no value), output:#14#14
- added U$271, U$356, U$441, U$526, U$611, U$696, U$781, U$866, U$951: (no value), output:#15#15
- added U$272, U$357, U$442, U$527, U$612, U$697, U$782, U$867, U$952: (no value), output:#16#16
- added U$273, U$358, U$443, U$528, U$613, U$698, U$783, U$868, U$953: (no value), output:#11#91420
- added U$274, U$359, U$444, U$529, U$614, U$699, U$784, U$869, U$954: (no value), output:#12#91420
- added U$275, U$360, U$445, U$530, U$615, U$700, U$785, U$870, U$955: (no value), output:#13#91420
- added U$276, U$361, U$446, U$531, U$616, U$701, U$786, U$871, U$956: (no value), output:#14#91420
- added U$277, U$362, U$447, U$532, U$617, U$702, U$787, U$872, U$957: (no value), output:#15#91420
- added U$278, U$363, U$448, U$533, U$618, U$703, U$788, U$873, U$958: (no value), output:#16#91420
- added U$279, U$364, U$449, U$534, U$619, U$704, U$789, U$874, U$959: (no value), output:#8#91421
- added U$280, U$365, U$450, U$535, U$620, U$705, U$790, U$875, U$960: (no value), output:#7#8
- added U$281, U$366, U$451, U$536, U$621, U$706, U$791, U$876, U$961: (no value), output:#6#8
- added U$282, U$367, U$452, U$537, U$622, U$707, U$792, U$877, U$962: (no value), output:#5#8
- added U$283, U$368, U$453, U$538, U$623, U$708, U$793, U$878, U$963: (no value), output:#4#8
- added U$284, U$369, U$454, U$539, U$624, U$709, U$794, U$879, U$964: (no value), output:#3#8
- added U$285, U$370, U$455, U$540, U$625, U$710, U$795, U$880, U$965: (no value), output:#2#8
- added U$286, U$371, U$456, U$541, U$626, U$711, U$796, U$881, U$966: (no value), output:#1#8
- added U$287, U$372, U$457, U$542, U$627, U$712, U$797, U$882, U$967: (no value), output:#0#8
- added U$288, U$373, U$458, U$543, U$628, U$713, U$798, U$883, U$968: (no value), output:#SHLD#9
- added U$289, U$374, U$459, U$544, U$629, U$714, U$799, U$884, U$969: (no value), output:#GND#10
- added U$290, U$375, U$460, U$545, U$630, U$715, U$800, U$885, U$970: (no value), output:#CHG#13
- added U$291, U$376, U$461, U$546, U$631, U$716, U$801, U$886, U$971: (no value), output:#PWR#14
- added U$292, U$377, U$462, U$547, U$632, U$717, U$802, U$887, U$972: (no value), output:#A0#18
- added U$293, U$378, U$463, U$548, U$633, U$718, U$803, U$888, U$973: (no value), output:USER0
- added U$294, U$379, U$464, U$549, U$634, U$719, U$804, U$889, U$974: (no value), output:#NC#2
- added U$295, U$380, U$465, U$550, U$635, U$720, U$805, U$890, U$975: (no value), output:#I2C#3
- added U$296, U$381, U$466, U$551, U$636, U$721, U$806, U$891, U$976: (no value), output:#SWD#501
- added U$297, U$382, U$467, U$552, U$637, U$722, U$807, U$892, U$977: (no value), output:#JP2#0
- added U$298, U$383, U$468, U$553, U$638, U$723, U$808, U$893, U$978: (no value), output:#LED_DO#0
- added U$299, U$384, U$469, U$554, U$639, U$724, U$809, U$894, U$979: (no value), output:#JP1#0
- added U$300, U$385, U$470, U$555, U$640, U$725, U$810, U$895, U$980: (no value), output:#9#10
- added U$301, U$386, U$471, U$556, U$641, U$726, U$811, U$896, U$981: (no value), output:#10#11
- added U$303, U$388, U$473, U$558, U$643, U$728, U$813, U$898, U$983: (no value), output:#18#18
- added U$304, U$389, U$474, U$559, U$644, U$729, U$814, U$899, U$984: (no value), output:##RESET##19
- added U$305, U$390, U$475, U$560, U$645, U$730, U$815, U$900, U$985: (no value), output:#NC#21
- added U$306, U$391, U$476, U$561, U$646, U$731, U$816, U$901, U$986: (no value), output:#G#22
- added U$307, U$392, U$477, U$562, U$647, U$732, U$817, U$902, U$987: (no value), output:#3V#23
- added U$308, U$393, U$478, U$563, U$648, U$733, U$818, U$903, U$988: (no value), output:#VU#23
- added U$310, U$395, U$480, U$565, U$650, U$735, U$820, U$905, U$990: (no value), output:#EN#27
- added U$311, U$396, U$481, U$566, U$651, U$736, U$821, U$906, U$991: (no value), output:#2#28
- added U$312, U$397, U$482, U$567, U$652, U$737, U$822, U$907, U$992: (no value), output:#3#28
- added U$313, U$398, U$483, U$568, U$653, U$738, U$823, U$908, U$993: (no value), output:#4#CS#28
- added U$314, U$399, U$484, U$569, U$654, U$739, U$824, U$909, U$994: (no value), output:#5#SCK#28
- added U$315, U$400, U$485, U$570, U$655, U$740, U$825, U$910, U$995: (no value), output:#6#PICO#28
- added U$316, U$401, U$486, U$571, U$656, U$741, U$826, U$911, U$996: (no value), output:#7#POCI#28
- added U$317, U$402, U$487, U$572, U$657, U$742, U$827, U$912, U$997: (no value), output:#8#RX1#A1#28
- added U$318, U$403, U$488, U$573, U$658, U$743, U$828, U$913, U$998: (no value), output:#9#TX1#A2#28
- added U$319, U$404, U$489, U$574, U$659, U$744, U$829, U$914, U$999: (no value), output:#10#28
- added U$341, U$426, U$511, U$596, U$681, U$766, U$851, U$936: (no value), output:CHG0
- added U$342, U$427, U$512, U$597, U$682, U$767, U$852, U$937: (no value), output:RESET0
- added U$343, U$428, U$513, U$598, U$683, U$768, U$853, U$938: (no value), output:#VUSB#0
- added U16, U21, U26, U31, U36, U41, U46, U51, U56: MCP73831, SparkFun-IC-Power:SOT23-5
- added U17, U22, U27, U32, U37, U42, U47, U52, U57: XC6222B331MR-G, SparkFun-IC-Power:SOT23-5
- added U18, U23, U28, U33, U38, U43, U48, U53, U58: UBLOX_NORA_W306, nora-w306:UBLOX-NORA-W3
- added U19, U24, U29, U34, U39, U44, U49, U54, U59: MAX17048, SparkFun-IC-Power:DFN-8
- added U20, U25, U30, U35, U40, U45, U50, U55, U60: CP2102N, SparkFun-IC-Comms:QFN24
- J14, J3, J8: value QWIIC_RA -> QWIIC_RIGHT_ANGLE
- R24, R51, R7: value 10k -> 100k
- U$100: device output:#1#4 -> output:#14#14
- U$101: device output:#13#13 -> output:#15#15
- U$102: device output:#14#14 -> output:#16#16
- U$103: device output:#15#15 -> output:#11#91420
- U$104: device output:#16#16 -> output:#12#91420
- U$105: device output:#11#91420 -> output:#13#91420
- U$106: device output:#12#91420 -> output:#14#91420
- U$107: device output:#13#91420 -> output:#15#91420
- U$108: device output:#14#91420 -> output:#16#91420
- U$109: device output:#15#91420 -> output:#8#91421
- U$11: device output:MA0 -> output:#SDPC#0
- U$110: device output:#16#91420 -> output:#7#8
- U$111: device output:#8#91421 -> output:#6#8
- U$112: device output:#7#8 -> output:#5#8
- U$113: device output:#6#8 -> output:#4#8
- U$114: device output:#5#8 -> output:#3#8
- U$115: device output:#4#8 -> output:#2#8
- U$116: device output:#3#8 -> output:#1#8
- U$117: device output:#2#8 -> output:#0#8
- U$118: device output:#1#8 -> output:#SHLD#9
- U$119: device output:#0#8 -> output:#GND#10
- U$120: device output:#SHLD#9 -> output:#CHG#13
- U$121: device output:#GND#10 -> output:#PWR#14
- U$122: device output:#CHG#13 -> output:#A0#18
- U$123: device output:#PWR#14 -> output:USER0
- U$124: device output:#A0#18 -> output:#NC#2
- U$125: device output:USER0 -> output:#I2C#3
- U$126: device output:#NC#2 -> output:#SWD#501
- U$127: device output:#I2C#3 -> output:#JP2#0
- U$128: device output:#SWD#501 -> output:#LED_DO#0
- U$129: device output:#JP2#0 -> output:#JP1#0
- U$130: device output:#LED_DO#0 -> output:#9#10
- U$131: device output:#JP1#0 -> output:#10#11
- U$132: device output:#9#10 -> output:#17#11
- U$133: device output:#10#11 -> output:#18#18
- U$134: device output:#17#11 -> output:##RESET##19
- U$135: device output:#18#18 -> output:#NC#21
- U$136: device output:##RESET##19 -> output:#G#22
- U$137: device output:#NC#21 -> output:#3V#23
- U$138: device output:#G#22 -> output:#VU#23
- U$139: device output:#3V#23 -> output:#VB26
- U$140: device output:#VU#23 -> output:#EN#27
- U$141: device output:#VB26 -> output:#2#28
- U$142: device output:#EN#27 -> output:#3#28
- U$143: device output:#2#28 -> output:#4#CS#28
- U$144: device output:#3#28 -> output:#5#SCK#28
- U$145: device output:#4#CS#28 -> output:#6#PICO#28
- U$146: device output:#5#SCK#28 -> output:#7#POCI#28
- U$147: device output:#6#PICO#28 -> output:#8#RX1#A1#28
- U$148: device output:#7#POCI#28 -> output:#9#TX1#A2#28
- U$149: device output:#8#RX1#A1#28 -> output:#10#28
- U$150: device output:#9#TX1#A2#28 -> output:#SDA#11#28
- U$151: device output:#10#28 -> output:#SCL#12#28
- U$152: device output:#SDA#11#28 -> output:#17#28
- U$153: device output:#SCL#12#28 -> output:#18#28
- U$154: device output:#17#28 -> SparkFun-Aesthetics:SFE_LOGO_FLAME_.1
- U$155: device output:#18#28 -> output:#LD#29
- U$156: device SparkFun-Aesthetics:SFE_LOGO_FLAME_.1 -> output:#VB26
- U$157: device output:#LD#29 -> output:#MEAS#1714141838
- U$158: device output:1830 -> output:THING_PLUS1714141839
- U$159: device output:RGB_14141832 -> output:NORA#W3061714141840
- U$160: device output:#VB26 -> output:#GND#ON#3061714141842
- U$161: device output:CUR1714141837 -> output:#17#11
- U$162: device output:#MEAS#1714141838 -> output:##RST##23061714141845
- U$163: device output:THING_PLUS1714141839 -> output:#JP3#23061714141846
- U$164: device output:NORA#W3061714141840 -> output:#100#23061714141846
- U$165: device output:#GND#ON#3061714141842 -> output:#500#23061714141846
- U$166: device output:23061714141843 -> output:IO180
- U$167: device output:#17#11 -> output:IO20
- U$168: device output:SDPC23061714141844 -> output:RGB_IO140
- U$169: device output:##RST##23061714141845 -> output:#CUR#0
- U$170: device output:#JP3#23061714141846 -> output:#SDPC#0
- U$171: device output:#100#23061714141846 -> output:CHG0
- U$172: device output:#500#23061714141846 -> output:RESET0
- U$173: device output:CHG0 -> output:#VUSB#0
- U$174: device output:RESET0 -> output:#EN#0
- U$175: device output:#VUSB#0 -> output:#3V3#0
- U$176: device output:#EN#0 -> output:THING_PLUS_0
- U$177: device output:#3V3#0 -> output:BOOT0
- U$178: device output:MA0 -> output:PWR0
- U$179: device output:THING_PLUS_0 -> output:NORA#W3060
- U$180: device output:BOOT0 -> SparkFun-Aesthetics:SFE_LOGO_FLAME_.2
- U$181: device output:PWR0 -> output:#A0#1
- U$182: device output:NORA#W3060 -> output:#0#4
- U$183: device SparkFun-Aesthetics:SFE_LOGO_FLAME_.2 -> output:#1#4
- U$184: device output:#A0#1 -> output:#13#13
- U$185: device output:#0#4 -> output:#14#14
- U$186: device output:#1#4 -> output:#15#15
- U$187: device output:#13#13 -> output:#16#16
- U$188: device output:#14#14 -> output:#11#91420
- U$189: device output:#15#15 -> output:#12#91420
- U$190: device output:#16#16 -> output:#13#91420
- U$191: device output:#11#91420 -> output:#14#91420
- U$192: device output:#12#91420 -> output:#15#91420
- U$193: device output:#13#91420 -> output:#16#91420
- U$194: device output:#14#91420 -> output:#8#91421
- U$195: device output:#15#91420 -> output:#7#8
- U$196: device output:#16#91420 -> output:#6#8
- U$197: device output:#8#91421 -> output:#5#8
- U$198: device output:#7#8 -> output:#4#8
- U$199: device output:#6#8 -> output:#3#8
- U$200: device output:#5#8 -> output:#2#8
- U$201: device output:#4#8 -> output:#1#8
- U$202: device output:#3#8 -> output:#0#8
- U$203: device output:#2#8 -> output:#SHLD#9
- U$204: device output:#1#8 -> output:#GND#10
- U$205: device output:#0#8 -> output:#CHG#13
- U$206: device output:#SHLD#9 -> output:#PWR#14
- U$207: device output:#GND#10 -> output:#A0#18
- U$208: device output:#CHG#13 -> output:USER0
- U$209: device output:#PWR#14 -> output:#NC#2
- U$21: device output:1830 -> output:RGB_IO140
- U$210: device output:#A0#18 -> output:#I2C#3
- U$211: device output:USER0 -> output:#SWD#501
- U$212: device output:#NC#2 -> output:#JP2#0
- U$213: device output:#I2C#3 -> output:#LED_DO#0
- U$214: device output:#SWD#501 -> output:#JP1#0
- U$215: device output:#JP2#0 -> output:#9#10
- U$216: device output:#LED_DO#0 -> output:#10#11
- U$217: device output:#JP1#0 -> output:#17#11
- U$218: device output:#9#10 -> output:#18#18
- U$219: device output:#10#11 -> output:##RESET##19
- U$220: device output:#17#11 -> output:#NC#21
- U$221: device output:#18#18 -> output:#G#22
- U$222: device output:##RESET##19 -> output:#3V#23
- U$223: device output:#NC#21 -> output:#VU#23
- U$224: device output:#G#22 -> output:#VB26
- U$225: device output:#3V#23 -> output:#EN#27
- U$226: device output:#VU#23 -> output:#2#28
- U$227: device output:#VB26 -> output:#3#28
- U$228: device output:#EN#27 -> output:#4#CS#28
- U$229: device output:#2#28 -> output:#5#SCK#28
- U$230: device output:#3#28 -> output:#6#PICO#28
- U$231: device output:#4#CS#28 -> output:#7#POCI#28
- U$232: device output:#5#SCK#28 -> output:#8#RX1#A1#28
- U$233: device output:#6#PICO#28 -> output:#9#TX1#A2#28
- U$234: device output:#7#POCI#28 -> output:#10#28
- U$235: device output:#8#RX1#A1#28 -> output:#SDA#11#28
- U$236: device output:#9#TX1#A2#28 -> output:#SCL#12#28
- U$237: device output:#10#28 -> output:#17#28
- U$238: device output:#SDA#11#28 -> output:#18#28
- U$239: device output:#SCL#12#28 -> SparkFun-Aesthetics:SFE_LOGO_FLAME_.1
- U$24: device output:RGB_14141832 -> output:#CUR#0
- U$240: device output:#17#28 -> output:#LD#29
- U$241: device output:#18#28 -> output:#VB26
- U$242: device SparkFun-Aesthetics:SFE_LOGO_FLAME_.1 -> output:#MEAS#1714141838
- U$243: device output:#LD#29 -> output:THING_PLUS1714141839
- U$244: device output:1830 -> output:NORA#W3061714141840
- U$245: device output:RGB_14141832 -> output:#GND#ON#3061714141842
- U$246: device output:#VB26 -> output:#17#11
- U$247: device output:CUR1714141837 -> output:##RST##23061714141845
- U$248: device output:#MEAS#1714141838 -> output:#JP3#23061714141846
- U$249: device output:THING_PLUS1714141839 -> output:#100#23061714141846
- U$250: device output:NORA#W3061714141840 -> output:#500#23061714141846
- U$251: device output:#GND#ON#3061714141842 -> output:IO180
- U$252: device output:23061714141843 -> output:IO20
- U$253: device output:#17#11 -> output:RGB_IO140
- U$254: device output:SDPC23061714141844 -> output:#CUR#0
- U$255: device output:##RST##23061714141845 -> output:#SDPC#0
- U$256: device output:#JP3#23061714141846 -> output:CHG0
- U$257: device output:#100#23061714141846 -> output:RESET0
- U$258: device output:#500#23061714141846 -> output:#VUSB#0
- U$27: device output:CUR1714141837 -> output:CHG0
- U$29: device output:23061714141843 -> output:RESET0
- U$34: device output:SDPC23061714141844 -> output:#VUSB#0
- U$4: device output:CHG0 -> output:IO180
- U$59: device output:#VUSB#0 -> output:#EN#0
- U$89: device output:#EN#0 -> output:#3V3#0
- U$9: device output:RESET0 -> output:IO20
- U$90: device output:#3V3#0 -> output:THING_PLUS_0
- U$92: device output:MA0 -> output:BOOT0
- U$93: device output:THING_PLUS_0 -> output:PWR0
- U$94: device output:BOOT0 -> output:NORA#W3060
- U$95: device output:PWR0 -> SparkFun-Aesthetics:SFE_LOGO_FLAME_.2
- U$96: device output:NORA#W3060 -> output:#A0#1
- U$97: device SparkFun-Aesthetics:SFE_LOGO_FLAME_.2 -> output:#0#4
- U$98: device output:#A0#1 -> output:#1#4
- U$99: device output:#0#4 -> output:#13#13
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Connections:
- new net !RESET!10: C132.1, J64.28, J66.10, Q52.3, S31.1, S31.2, U53.J3
- new net !RESET!11: C144.1, J70.28, J72.10, Q57.3, S34.1, S34.2, U58.J3
- new net !RESET!3: C48.1, J22.28, J24.10, Q17.3, S10.1, S10.2, U18.J3
- new net !RESET!4: C60.1, J28.28, J30.10, Q22.3, S13.1, S13.2, U23.J3
- new net !RESET!5: C72.1, J34.28, J36.10, Q27.3, S16.1, S16.2, U28.J3
- new net !RESET!6: C84.1, J40.28, J42.10, Q32.3, S19.1, S19.2, U33.J3
- new net !RESET!7: C96.1, J46.28, J48.10, Q37.3, S22.1, S22.2, U38.J3
- new net !RESET!8: C108.1, J52.28, J54.10, Q42.3, S25.1, S25.2, U43.J3
- new net !RESET!9: C120.1, J58.28, J60.10, Q47.3, S28.1, S28.2, U48.J3
- new net 3.3V10: C122.1, C125.1, C128.1, I2C10.2, J62.2, J64.27, J66.1, JP33.1, LED10.1, Q53.2, Q54.2, R270.1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
- new net 3.3V11: C134.1, C137.1, C140.1, I2C11.2, J68.2, J70.27, J72.1, JP36.1, LED11.1, Q58.2, Q59.2, R295.1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
- new net 3.3V3: C38.1, C41.1, C44.1, I2C3.2, J20.2, J22.27, J24.1, JP12.1, LED3.1, Q18.2, Q19.2, R95.1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
- new net 3.3V4: C50.1, C53.1, C56.1, I2C4.2, J26.2, J28.27, J30.1, JP15.1, LED4.1, Q23.2, Q24.2, R120.1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
- new net 3.3V5: C62.1, C65.1, C68.1, I2C5.2, J32.2, J34.27, J36.1, JP18.1, LED5.1, Q28.2, Q29.2, R145.1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
- new net 3.3V6: C74.1, C77.1, C80.1, I2C6.2, J38.2, J40.27, J42.1, JP21.1, LED6.1, Q33.2, Q34.2, R170.1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
- new net 3.3V7: C86.1, C89.1, C92.1, I2C7.2, J44.2, J46.27, J48.1, JP24.1, LED7.1, Q38.2, Q39.2, R195.1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
- new net 3.3V8: C101.1, C104.1, C98.1, I2C8.2, J50.2, J52.27, J54.1, JP27.1, LED8.1, Q43.2, Q44.2, R220.1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
- new net 3.3V9: C110.1, C113.1, C116.1, I2C9.2, J56.2, J58.27, J60.1, JP30.1, LED9.1, Q48.2, Q49.2, R245.1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
- new net CC10: J27.A5, R110.2
- new net CC11: J33.B5, R134.2
- new net CC12: J33.A5, R135.2
- new net CC13: J39.B5, R159.2
- new net CC14: J39.A5, R160.2
- new net CC15: J45.B5, R184.2
- new net CC16: J45.A5, R185.2
- new net CC17: J51.B5, R209.2
- new net CC18: J51.A5, R210.2
- new net CC19: J57.B5, R234.2
- new net CC20: J57.A5, R235.2
- new net CC21: J63.B5, R259.2
- new net CC22: J63.A5, R260.2
- new net CC23: J69.B5, R284.2
- new net CC24: J69.A5, R285.2
- new net CC7: J21.B5, R84.2
- new net CC8: J21.A5, R85.2
- new net CC9: J27.B5, R109.2
- new net CHG10: CHG10.2, U51.1
- new net CHG11: CHG11.2, U56.1
- new net CHG3: CHG3.2, U16.1
- new net CHG4: CHG4.2, U21.1
- new net CHG5: CHG5.2, U26.1
- new net CHG6: CHG6.2, U31.1
- new net CHG7: CHG7.2, U36.1
- new net CHG8: CHG8.2, U41.1
- new net CHG9: CHG9.2, U46.1
- new net DTR10: Q52.1, R264.1, U55.23
- new net DTR11: Q57.1, R289.1, U60.23
- new net DTR3: Q17.1, R89.1, U20.23
- new net DTR4: Q22.1, R114.1, U25.23
- new net DTR5: Q27.1, R139.1, U30.23
- new net DTR6: Q32.1, R164.1, U35.23
- new net DTR7: Q37.1, R189.1, U40.23
- new net DTR8: Q42.1, R214.1, U45.23
- new net DTR9: Q47.1, R239.1, U50.23
- new net EN10: J64.11, R256.2, U52.3
- new net EN11: J70.11, R281.2, U57.3
- new net EN3: J22.11, R81.2, U17.3
- new net EN4: J28.11, R106.2, U22.3
- new net EN5: J34.11, R131.2, U27.3
- new net EN6: J40.11, R156.2, U32.3
- new net EN7: J46.11, R181.2, U37.3
- new net EN8: J52.11, R206.2, U42.3
- new net EN9: J58.11, R231.2, U47.3
- new net GND10: C121.2, C122.2, C123.2, C124.2, C125.2, C126.2, C127.2, C128.2, C129.2, C130.2, C131.2, C132.2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
- new net GND11: C133.2, C134.2, C135.2, C136.2, C137.2, C138.2, C139.2, C140.2, C141.2, C142.2, C143.2, C144.2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
- new net GND3: C37.2, C38.2, C39.2, C40.2, C41.2, C42.2, C43.2, C44.2, C45.2, C46.2, C47.2, C48.2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
- new net GND4: C49.2, C50.2, C51.2, C52.2, C53.2, C54.2, C55.2, C56.2, C57.2, C58.2, C59.2, C60.2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
- new net GND5: C61.2, C62.2, C63.2, C64.2, C65.2, C66.2, C67.2, C68.2, C69.2, C70.2, C71.2, C72.2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
- new net GND6: C73.2, C74.2, C75.2, C76.2, C77.2, C78.2, C79.2, C80.2, C81.2, C82.2, C83.2, C84.2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
- new net GND7: C85.2, C86.2, C87.2, C88.2, C89.2, C90.2, C91.2, C92.2, C93.2, C94.2, C95.2, C96.2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
- new net GND8: C100.2, C101.2, C102.2, C103.2, C104.2, C105.2, C106.2, C107.2, C108.2, C97.2, C98.2, C99.2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
- new net GND9: C109.2, C110.2, C111.2, C112.2, C113.2, C114.2, C115.2, C116.2, C117.2, C118.2, C119.2, C120.2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
- new net N$100: R82.1, R83.2, U20.8
- new net N$101: CUR3.2, U16.5
- new net N$102: CUR3.1, R86.1
- new net N$103: CUR3.3, R78.2
- new net N$104: Q16.1, R87.2
- new net N$105: R88.2, S11.3, S11.4
- new net N$106: Q17.5, R89.2
- new net N$107: Q17.2, R90.2
- new net N$108: LED3.2, R91.1
- new net N$109: D22.A, R91.2
- new net N$110: D23.6, U20.3
- new net N$111: D23.1, J21.A6, J21.B6
- new net N$112: D23.4, U20.4
- new net N$113: D23.3, J21.A7, J21.B7
- new net N$114: CHG3.1, D20.C
- new net N$115: D24.DI, JP10.2
- new net N$116: I2C3.3, R92.2
- new net N$117: I2C3.1, R93.2
- new net N$118: JP11.2, R80.1
- new net N$119: D19.C, MEAS3.1, MEAS3.3, Q16.2
- new net N$120: Q18.1, R94.2
- new net N$121: C45.1, J23.4, Q18.3, R96.1
- new net N$122: R94.1, R95.2, SDPC3.2
- new net N$123: Q20.3, R97.2, R98.2
- new net N$124: C42.1, C43.1, Q19.3, R79.1, U20.5, U20.6, U20.7
- new net N$125: C46.1, D24.VCC, JP12.2
- new net N$126: Q19.1, R98.1
- new net N$127: R99.1, SDPC3.3
- new net N$128: Q20.1, R100.2
- new net N$129: D26.A, R102.2
- new net N$130: R104.2, U25.9
- new net N$131: D27.A, R105.2
- new net N$132: R107.1, R108.2, U25.8
- new net N$133: CUR4.2, U21.5
- new net N$134: CUR4.1, R111.1
- new net N$135: CUR4.3, R103.2
- new net N$136: Q21.1, R112.2
- new net N$137: R113.2, S14.3, S14.4
- new net N$138: Q22.5, R114.2
- new net N$139: Q22.2, R115.2
- new net N$140: LED4.2, R116.1
- new net N$141: D28.A, R116.2
- new net N$142: D29.6, U25.3
- new net N$143: D29.1, J27.A6, J27.B6
- new net N$144: D29.4, U25.4
- new net N$145: D29.3, J27.A7, J27.B7
- new net N$146: CHG4.1, D26.C
- new net N$147: D30.DI, JP13.2
- new net N$148: I2C4.3, R117.2
- new net N$149: I2C4.1, R118.2
- new net N$150: JP14.2, R105.1
- new net N$151: D25.C, MEAS4.1, MEAS4.3, Q21.2
- new net N$152: Q23.1, R119.2
- new net N$153: C57.1, J29.4, Q23.3, R121.1
- new net N$154: R119.1, R120.2, SDPC4.2
- new net N$155: Q25.3, R122.2, R123.2
- new net N$156: C54.1, C55.1, Q24.3, R104.1, U25.5, U25.6, U25.7
- new net N$157: C58.1, D30.VCC, JP15.2
- new net N$158: Q24.1, R123.1
- new net N$159: R124.1, SDPC4.3
- new net N$160: Q25.1, R125.2
- new net N$161: D32.A, R127.2
- new net N$162: R129.2, U30.9
- new net N$163: D33.A, R130.2
- new net N$164: R132.1, R133.2, U30.8
- new net N$165: CUR5.2, U26.5
- new net N$166: CUR5.1, R136.1
- new net N$167: CUR5.3, R128.2
- new net N$168: Q26.1, R137.2
- new net N$169: R138.2, S17.3, S17.4
- new net N$170: Q27.5, R139.2
- new net N$171: Q27.2, R140.2
- new net N$172: LED5.2, R141.1
- new net N$173: D34.A, R141.2
- new net N$174: D35.6, U30.3
- new net N$175: D35.1, J33.A6, J33.B6
- new net N$176: D35.4, U30.4
- new net N$177: D35.3, J33.A7, J33.B7
- new net N$178: CHG5.1, D32.C
- new net N$179: D36.DI, JP16.2
- new net N$180: I2C5.3, R142.2
- new net N$181: I2C5.1, R143.2
- new net N$182: JP17.2, R130.1
- new net N$183: D31.C, MEAS5.1, MEAS5.3, Q26.2
- new net N$184: Q28.1, R144.2
- new net N$185: C69.1, J35.4, Q28.3, R146.1
- new net N$186: R144.1, R145.2, SDPC5.2
- new net N$187: Q30.3, R147.2, R148.2
- new net N$188: C66.1, C67.1, Q29.3, R129.1, U30.5, U30.6, U30.7
- new net N$189: C70.1, D36.VCC, JP18.2
- new net N$190: Q29.1, R148.1
- new net N$191: R149.1, SDPC5.3
- new net N$192: Q30.1, R150.2
- new net N$193: D38.A, R152.2
- new net N$194: R154.2, U35.9
- new net N$195: D39.A, R155.2
- new net N$196: R157.1, R158.2, U35.8
- new net N$197: CUR6.2, U31.5
- new net N$198: CUR6.1, R161.1
- new net N$199: CUR6.3, R153.2
- new net N$200: Q31.1, R162.2
- new net N$201: R163.2, S20.3, S20.4
- new net N$202: Q32.5, R164.2
- new net N$203: Q32.2, R165.2
- new net N$204: LED6.2, R166.1
- new net N$205: D40.A, R166.2
- new net N$206: D41.6, U35.3
- new net N$207: D41.1, J39.A6, J39.B6
- new net N$208: D41.4, U35.4
- new net N$209: D41.3, J39.A7, J39.B7
- new net N$210: CHG6.1, D38.C
- new net N$211: D42.DI, JP19.2
- new net N$212: I2C6.3, R167.2
- new net N$213: I2C6.1, R168.2
- new net N$214: JP20.2, R155.1
- new net N$215: D37.C, MEAS6.1, MEAS6.3, Q31.2
- new net N$216: Q33.1, R169.2
- new net N$217: C81.1, J41.4, Q33.3, R171.1
- new net N$218: R169.1, R170.2, SDPC6.2
- new net N$219: Q35.3, R172.2, R173.2
- new net N$220: C78.1, C79.1, Q34.3, R154.1, U35.5, U35.6, U35.7
- new net N$221: C82.1, D42.VCC, JP21.2
- new net N$222: Q34.1, R173.1
- new net N$223: R174.1, SDPC6.3
- new net N$224: Q35.1, R175.2
- new net N$225: D44.A, R177.2
- new net N$226: R179.2, U40.9
- new net N$227: D45.A, R180.2
- new net N$228: R182.1, R183.2, U40.8
- new net N$229: CUR7.2, U36.5
- new net N$230: CUR7.1, R186.1
- new net N$231: CUR7.3, R178.2
- new net N$232: Q36.1, R187.2
- new net N$233: R188.2, S23.3, S23.4
- new net N$234: Q37.5, R189.2
- new net N$235: Q37.2, R190.2
- new net N$236: LED7.2, R191.1
- new net N$237: D46.A, R191.2
- new net N$238: D47.6, U40.3
- new net N$239: D47.1, J45.A6, J45.B6
- new net N$240: D47.4, U40.4
- new net N$241: D47.3, J45.A7, J45.B7
- new net N$242: CHG7.1, D44.C
- new net N$243: D48.DI, JP22.2
- new net N$244: I2C7.3, R192.2
- new net N$245: I2C7.1, R193.2
- new net N$246: JP23.2, R180.1
- new net N$247: D43.C, MEAS7.1, MEAS7.3, Q36.2
- new net N$248: Q38.1, R194.2
- new net N$249: C93.1, J47.4, Q38.3, R196.1
- new net N$250: R194.1, R195.2, SDPC7.2
- new net N$251: Q40.3, R197.2, R198.2
- new net N$252: C90.1, C91.1, Q39.3, R179.1, U40.5, U40.6, U40.7
- new net N$253: C94.1, D48.VCC, JP24.2
- new net N$254: Q39.1, R198.1
- new net N$255: R199.1, SDPC7.3
- new net N$256: Q40.1, R200.2
- new net N$257: D50.A, R202.2
- new net N$258: R204.2, U45.9
- new net N$259: D51.A, R205.2
- new net N$260: R207.1, R208.2, U45.8
- new net N$261: CUR8.2, U41.5
- new net N$262: CUR8.1, R211.1
- new net N$263: CUR8.3, R203.2
- new net N$264: Q41.1, R212.2
- new net N$265: R213.2, S26.3, S26.4
- new net N$266: Q42.5, R214.2
- new net N$267: Q42.2, R215.2
- new net N$268: LED8.2, R216.1
- new net N$269: D52.A, R216.2
- new net N$270: D53.6, U45.3
- new net N$271: D53.1, J51.A6, J51.B6
- new net N$272: D53.4, U45.4
- new net N$273: D53.3, J51.A7, J51.B7
- new net N$274: CHG8.1, D50.C
- new net N$275: D54.DI, JP25.2
- new net N$276: I2C8.3, R217.2
- new net N$277: I2C8.1, R218.2
- new net N$278: JP26.2, R205.1
- new net N$279: D49.C, MEAS8.1, MEAS8.3, Q41.2
- new net N$280: Q43.1, R219.2
- new net N$281: C105.1, J53.4, Q43.3, R221.1
- new net N$282: R219.1, R220.2, SDPC8.2
- new net N$283: Q45.3, R222.2, R223.2
- new net N$284: C102.1, C103.1, Q44.3, R204.1, U45.5, U45.6, U45.7
- new net N$285: C106.1, D54.VCC, JP27.2
- new net N$286: Q44.1, R223.1
- new net N$287: R224.1, SDPC8.3
- new net N$288: Q45.1, R225.2
- new net N$289: D56.A, R227.2
- new net N$290: R229.2, U50.9
- new net N$291: D57.A, R230.2
- new net N$292: R232.1, R233.2, U50.8
- new net N$293: CUR9.2, U46.5
- new net N$294: CUR9.1, R236.1
- new net N$295: CUR9.3, R228.2
- new net N$296: Q46.1, R237.2
- new net N$297: R238.2, S29.3, S29.4
- new net N$298: Q47.5, R239.2
- new net N$299: Q47.2, R240.2
- new net N$300: LED9.2, R241.1
- new net N$301: D58.A, R241.2
- new net N$302: D59.6, U50.3
- new net N$303: D59.1, J57.A6, J57.B6
- new net N$304: D59.4, U50.4
- new net N$305: D59.3, J57.A7, J57.B7
- new net N$306: CHG9.1, D56.C
- new net N$307: D60.DI, JP28.2
- new net N$308: I2C9.3, R242.2
- new net N$309: I2C9.1, R243.2
- new net N$310: JP29.2, R230.1
- new net N$311: D55.C, MEAS9.1, MEAS9.3, Q46.2
- new net N$312: Q48.1, R244.2
- new net N$313: C117.1, J59.4, Q48.3, R246.1
- new net N$314: R244.1, R245.2, SDPC9.2
- new net N$315: Q50.3, R247.2, R248.2
- new net N$316: C114.1, C115.1, Q49.3, R229.1, U50.5, U50.6, U50.7
- new net N$317: C118.1, D60.VCC, JP30.2
- new net N$318: Q49.1, R248.1
- new net N$319: R249.1, SDPC9.3
- new net N$320: Q50.1, R250.2
- new net N$321: D62.A, R252.2
- new net N$322: R254.2, U55.9
- new net N$323: D63.A, R255.2
- new net N$324: R257.1, R258.2, U55.8
- new net N$325: CUR10.2, U51.5
- new net N$326: CUR10.1, R261.1
- new net N$327: CUR10.3, R253.2
- new net N$328: Q51.1, R262.2
- new net N$329: R263.2, S32.3, S32.4
- new net N$330: Q52.5, R264.2
- new net N$331: Q52.2, R265.2
- new net N$332: LED10.2, R266.1
- new net N$333: D64.A, R266.2
- new net N$334: D65.6, U55.3
- new net N$335: D65.1, J63.A6, J63.B6
- new net N$336: D65.4, U55.4
- new net N$337: D65.3, J63.A7, J63.B7
- new net N$338: CHG10.1, D62.C
- new net N$339: D66.DI, JP31.2
- new net N$340: I2C10.3, R267.2
- new net N$341: I2C10.1, R268.2
- new net N$342: JP32.2, R255.1
- new net N$343: D61.C, MEAS10.1, MEAS10.3, Q51.2
- new net N$344: Q53.1, R269.2
- new net N$345: C129.1, J65.4, Q53.3, R271.1
- new net N$346: R269.1, R270.2, SDPC10.2
- new net N$347: Q55.3, R272.2, R273.2
- new net N$348: C126.1, C127.1, Q54.3, R254.1, U55.5, U55.6, U55.7
- new net N$349: C130.1, D66.VCC, JP33.2
- new net N$350: Q54.1, R273.1
- new net N$351: R274.1, SDPC10.3
- new net N$352: Q55.1, R275.2
- new net N$353: D68.A, R277.2
- new net N$354: R279.2, U60.9
- new net N$355: D69.A, R280.2
- new net N$356: R282.1, R283.2, U60.8
- new net N$357: CUR11.2, U56.5
- new net N$358: CUR11.1, R286.1
- new net N$359: CUR11.3, R278.2
- new net N$360: Q56.1, R287.2
- new net N$361: R288.2, S35.3, S35.4
- new net N$362: Q57.5, R289.2
- new net N$363: Q57.2, R290.2
- new net N$364: LED11.2, R291.1
- new net N$365: D70.A, R291.2
- new net N$366: D71.6, U60.3
- new net N$367: D71.1, J69.A6, J69.B6
- new net N$368: D71.4, U60.4
- new net N$369: D71.3, J69.A7, J69.B7
- new net N$370: CHG11.1, D68.C
- new net N$371: D72.DI, JP34.2
- new net N$372: I2C11.3, R292.2
- new net N$373: I2C11.1, R293.2
- new net N$374: JP35.2, R280.1
- new net N$375: D67.C, MEAS11.1, MEAS11.3, Q56.2
- new net N$376: Q58.1, R294.2
- new net N$377: C141.1, J71.4, Q58.3, R296.1
- new net N$378: R294.1, R295.2, SDPC11.2
- new net N$379: Q60.3, R297.2, R298.2
- new net N$380: C138.1, C139.1, Q59.3, R279.1, U60.5, U60.6, U60.7
- new net N$381: C142.1, D72.VCC, JP36.2
- new net N$382: Q59.1, R298.1
- new net N$383: R299.1, SDPC11.3
- new net N$384: Q60.1, R300.2
- new net N$97: D20.A, R77.2
- new net N$98: R79.2, U20.9
- new net N$99: D21.A, R80.2
- new net PA17: J22.4, JP10.1, U18.J9
- new net PA18: J22.3, U18.J8
- new net PA19: J22.6, U18.H9
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Routing:
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- added copper zone on layer 1, net 3.3V10
- added copper zone on layer 15, net 3.3V10
- added copper zone on layer 1, net 3.3V11
- added copper zone on layer 15, net 3.3V11
- added copper zone on layer 1, net 3.3V3
- added copper zone on layer 15, net 3.3V3
- added copper zone on layer 1, net 3.3V4
- added copper zone on layer 15, net 3.3V4
- added copper zone on layer 1, net 3.3V5
- added copper zone on layer 15, net 3.3V5
- added copper zone on layer 1, net 3.3V6
- added copper zone on layer 15, net 3.3V6
- added copper zone on layer 1, net 3.3V7
- added copper zone on layer 15, net 3.3V7
- added copper zone on layer 1, net 3.3V8
- added copper zone on layer 15, net 3.3V8
- added copper zone on layer 1, net 3.3V9
- added copper zone on layer 15, net 3.3V9
- added copper zone on layer 1, net GND10
- added copper zone on layer 16, net GND10
- added copper zone on layer 2, net GND10
- added copper zone on layer 1, net GND11
- added copper zone on layer 16, net GND11
- added copper zone on layer 2, net GND11
- added copper zone on layer 1, net GND3
- added copper zone on layer 16, net GND3
- added copper zone on layer 2, net GND3
- added copper zone on layer 1, net GND4
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Other:
- board size 83.3 x 80.3 mm -> 106.7 x 203.2 mm
- board text added: "v10"
- board text removed: "v05"
